File: xmosio2.sch (EAGLE design)
At the start: 103 parts, among them IC1 IDTQS3245QSOP20, IC2 IDTQS3245QSOP20, IC3 IDTQS3245QSOP20, IC4 IDTQS3245QSOP20, IC5 IDTQS3245QSOP20, U1 24 MHz Osc. (F535L-24), U2 USD-SOCKETNEW, X1 0446200002, X2 MINI-USB-UX60-MB-5S8

Commit message: Latest revision. Fixes:  - Rename the power line from 4.1 to 4.3v  - Make +5v be the only one with a specified width to aid in routing. The PCB traces are sufficiently wide, given they’re in air, and there are multiple supplies to the main chip  - Added the required vias on the ground pad of the XMOS chip  - Make LEDs be 0805 rather than 0603  - Fixes identified by Xcore.com user eez-open  - Fix connection of 1v converter EN to +5V  - Route JTAG lines and make Link lines pass DRC  - Add an SD card  - Add LEDs for debugging later  - Add a switch so that firmware can be booted from a golden master, rather than the latest on-board
Parts:
- removed C33: 100nF, rcl:C-EUC0603
- removed LED5: (no value), SparkFun-LED:LED0603
- removed R16, R17: 10K, rcl:R-EU_R0603
- added C46: 100nF, rcl:C-EUC0603
- added LED6: ok33, led:LEDCHIP-LED0805
- added R27: 47K, rcl:R-EU_R0603
- added S2: FLASH_MODE, SparkFun:TAC_SWITCHPTH
- LED2, LED3, LED4: value (none) -> ok33; device SparkFun-LED:LED0603 -> led:LEDCHIP-LED0805
Connections:
- net +4.1V renamed +4.3V
- new net EN_1V0: R27.1, U$5.EN@5, U$6.!RESET!@1
- net +5V: no longer U$5.EN@5, U$6.!RESET!@1
- net GND: now also C46.2, S2.3, S2.4; no longer C33.2, R15.2, R16.2, R17.2
- net LED0: now also LED6.A; no longer LED2.A
- net LED1: now also LED2.A; no longer LED3.A
- net LED2: now also LED3.A; no longer LED4.A
- net LED3: now also LED4.A; no longer LED5.A
- net N$10: now also LED1.C; no longer LED1.A
- net N$24: now also LED4.C; no longer LED5.C
- net N$25: now also LED3.C; no longer LED4.C
- net N$26: now also LED2.C; no longer LED3.C
- net N$27: now also LED6.C; no longer LED2.C
- net N$33: now also R15.1, S2.1, S2.2
- net SD_ADQ2/QS_D0: no longer R15.1
- net SD_ADQ3/QS_D1: no longer R16.1
- net SD_ADQ4/QS_D2: no longer R17.1
- net VCCINT: no longer C33.1, U$6.VCC@6
- net VCCIO: now also C46.1, LED1.A, R15.2, R27.2, U$6.VCC@6; no longer LED1.C
Other:
- note added: "Note: SDRAM byte lanes aren't supported. Do a read/modify/write to write individual bytes"
- note removed: "Pull-downs to ensure boot from QSPI"
- moved on the sheet: C27, C28, C29, C31, C32, C34, C35, C36, C37, C38, C39, C40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

Commit message: Tidy up the board labelling
Parts:
- renumbered LED2 to DBG1, LED3 to DBG2, LED4 to DBG3, LED6 to DBG0, S1 to RESET_SW, S2 to BOOT_SW, X2 to USBPOWER
Changed lines of the file:
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@@
 <setting verticaltext="up"/>
 </settings>
-<grid distance="0.1" unitdist="inch" unit="inch" style="lines" multiple="1" display="yes" altdistance="0.01" altunitdist="inch" altunit="inch"/>
+<grid distance="0.1" unitdist="inch" unit="inch" style="lines" multiple="1" display="no" altdistance="0.01" altunitdist="inch" altunit="inch"/>
 <layers>
 <layer number="1" name="Top" color="4" fill="1" visible="no" active="no"/>
@@
 <part name="C44" library="rcl" deviceset="C-EU" device="C0603" value="10nF"/>
 <part name="GND36" library="supply1" deviceset="GND" device=""/>
-<part name="S1" library="SparkFun" deviceset="TAC_SWITCH" device="PTH" value="MANUAL_RESET"/>
+<part name="RESET_SW" library="SparkFun" deviceset="TAC_SWITCH" device="PTH" value="MANUAL_RESET"/>
 <part name="GND37" library="supply1" deviceset="GND" device=""/>
 <part name="FRAME1" library="frames" deviceset="A3L-LOC" device="" value="BUS I/O"/>
@@
 <part name="GND45" library="supply1" deviceset="GND" device=""/>
 <part name="P+4" library="supply1" deviceset="+5V" device=""/>
-<part name="X2" library="con-hirose" deviceset="MINI-USB-" device="UX60-MB-5S8"/>
+<part name="USBPOWER" library="con-hirose" deviceset="MINI-USB-" device="UX60-MB-5S8"/>
 <part name="R20" library="rcl" deviceset="R-EU_" device="R0603" value="1K"/>
 <part name="R21" library="rcl" deviceset="R-EU_" device="R0603" value="1K"/>
@@
 <part name="R27" library="rcl" deviceset="R-EU_" device="R0603" value="47K"/>
 <part name="C46" library="rcl" deviceset="C-EU" device="C0603" value="100nF"/>
-<part name="LED6" library="led" deviceset="LED" device="CHIP-LED0805" value="ok33"/>
-<part name="LED2" library="led" deviceset="LED" device="CHIP-LED0805" value="ok33"/>
-<part name="LED3" library="led" deviceset="LED" device="CHIP-LED0805" value="ok33"/>
-<part name="LED4" library="led" deviceset="LED" device="CHIP-LED0805" value="ok33"/>
+<part name="DBG0" library="led" deviceset="LED" device="CHIP-LED0805" value="ok33"/>
+<part name="DBG1" library="led" deviceset="LED" device="CHIP-LED0805" value="ok33"/>
+<part name="DBG2" library="led" deviceset="LED" device="CHIP-LED0805" value="ok33"/>
+<part name="DBG3" library="led" deviceset="LED" device="CHIP-LED0805" value="ok33"/>
 <part name="U$13" library="sjg-power" deviceset="+4.3V" device=""/>
 <part name="U$14" library="sjg-power" deviceset="+4.3V" device=""/>
@@
 <part name="VCC23" library="supply1" deviceset="VCCIO" device=""/>
 <part name="VCC24" library="supply1" deviceset="VCCIO" device=""/>
-<part name="S2" library="SparkFun" deviceset="TAC_SWITCH" device="PTH" value="FLASH_MODE"/>
+<part name="BOOT_SW" library="SparkFun" deviceset="TAC_SWITCH" device="PTH" value="FLASH_MODE"/>
 <part name="GND38" library="supply1" deviceset="GND" device=""/>
 <part name="R15" library="rcl" deviceset="R-EU_" device="R0603" value="10K"/>
@@
 <instance part="GND45" gate="1" x="-17.78" y="58.42"/>
 <instance part="P+4" gate="1" x="-17.78" y="81.28"/>
-<instance part="X2" gate="G$1" x="-7.62" y="68.58"/>
+<instance part="USBPOWER" gate="G$1" x="-7.62" y="68.58"/>
 <instance part="GND48" gate="1" x="281.94" y="-63.5"/>
 <instance part="R27" gate="G$1" x="302.26" y="-50.8" rot="R90"/>
@@
 </segment>
 <segment>
-<pinref part="X2" gate="G$1" pin="5"/>
+<pinref part="USBPOWER" gate="G$1" pin="5"/>
 <pinref part="GND45" gate="1" pin="GND"/>
 <wire x1="-12.7" y1="63.5" x2="-17.78" y2="63.5" width="0.1524" layer="91"/>
@@
 </segment>
 <segment>
-<pinref part="X2" gate="G$1" pin="1"/>
+<pinref part="USBPOWER" gate="G$1" pin="1"/>
 <pinref part="P+4" gate="1" pin="+5V"/>
 <wire x1="-12.7" y1="73.66" x2="-17.78" y2="73.66" width="0.1524" layer="91"/>
@@
 </instance>
 <instance part="FRAME3" gate="G$1" x="-58.42" y="-129.54"/>
-<instance part="S2" gate="S" x="35.56" y="-5.08" smashed="yes">
-<attribute name="NAME" x="34.29" y="0" size="1.778" layer="95"/>
-<attribute name="VALUE" x="27.94" y="3.81" size="2.1844" layer="96"/>
+<instance part="BOOT_SW" gate="S" x="35.56" y="-5.08" smashed="yes">
+<attribute name="NAME" x="31.75" y="0" size="1.778" layer="95"/>
+<attribute name="VALUE" x="30.48" y="-19.05" size="2.1844" layer="96"/>
 </instance>
 <instance part="GND38" gate="1" x="45.72" y="-12.7"/>
@@
 </segment>
 <segment>
-<pinref part="S2" gate="S" pin="3"/>
-<pinref part="S2" gate="S" pin="4"/>
+<pinref part="BOOT_SW" gate="S" pin="3"/>
+<pinref part="BOOT_SW" gate="S" pin="4"/>
 <wire x1="40.64" y1="-5.08" x2="40.64" y2="-7.62" width="0.1524" layer="91"/>
 <pinref part="GND38" gate="1" pin="GND"/>
@@
 <segment>
 <pinref part="U$2" gate="TILE0" pin="X0D39@6"/>
-<pinref part="S2" gate="S" pin="2"/>
+<pinref part="BOOT_SW" gate="S" pin="2"/>
 <wire x1="30.48" y1="-7.62" x2="20.32" y2="-7.62" width="0.1524" layer="91"/>
-<pinref part="S2" gate="S" pin="1"/>
+<pinref part="BOOT_SW" gate="S" pin="1"/>
 <wire x1="20.32" y1="-7.62" x2="-12.7" y2="-7.62" width="0.1524" layer="91"/>
 <wire x1="30.48" y1="-7.62" x2="30.48" y2="-5.08" width="0.1524" layer="91"/>
@@
 <instance part="C44" gate="G$1" x="254" y="101.6" rot="R90"/>
 <instance part="GND36" gate="1" x="246.38" y="93.98"/>
-<instance part="S1" gate="S" x="287.02" y="104.14" smashed="yes">
+<instance part="RESET_SW" gate="S" x="287.02" y="104.14" smashed="yes">
 <attribute name="NAME" x="284.48" y="110.49" size="1.778" layer="95"/>
-<attribute name="VALUE" x="276.86" y="113.03" size="2.1844" layer="96"/>
+<attribute name="VALUE" x="276.86" y="87.63" size="2.1844" layer="96"/>
 </instance>
 <instance part="GND37" gate="1" x="297.18" y="93.98"/>
@@
 </segment>
 <segment>
-<pinref part="S1" gate="S" pin="4"/>
+<pinref part="RESET_SW" gate="S" pin="4"/>
 <pinref part="GND37" gate="1" pin="GND"/>
 <wire x1="292.1" y1="101.6" x2="297.18" y2="101.6" width="0.1524" layer="91"/>
 <wire x1="297.18" y1="101.6" x2="297.18" y2="96.52" width="0.1524" layer="91"/>
-<pinref part="S1" gate="S" pin="3"/>
+<pinref part="RESET_SW" gate="S" pin="3"/>
 <wire x1="292.1" y1="104.14" x2="297.18" y2="104.14" width="0.1524" layer="91"/>
 <wire x1="297.18" y1="104.14" x2="297.18" y2="101.6" width="0.1524" layer="91"/>
@@
 <pinref part="C44" gate="G$1" pin="2"/>
 <wire x1="269.24" y1="101.6" x2="259.08" y2="101.6" width="0.1524" layer="91"/>
-<pinref part="S1" gate="S" pin="2"/>
+<pinref part="RESET_SW" gate="S" pin="2"/>
 <wire x1="269.24" y1="101.6" x2="276.86" y2="101.6" width="0.1524" layer="91"/>
 <junction x="269.24" y="101.6"/>
-<pinref part="S1" gate="S" pin="1"/>
+<pinref part="RESET_SW" gate="S" pin="1"/>
 <wire x1="276.86" y1="101.6" x2="281.94" y2="101.6" width="0.1524" layer="91"/>
 <wire x1="276.86" y1="101.6" x2="276.86" y2="104.14" width="0.1524" layer="91"/>
@@
 <attribute name="VALUE" x="270.51" y="81.28" size="1.778" layer="96"/>
 </instance>
-<instance part="LED6" gate="G$1" x="91.44" y="106.68" rot="R90"/>
-<instance part="LED2" gate="G$1" x="91.44" y="96.52" rot="R90"/>
-<instance part="LED3" gate="G$1" x="91.44" y="86.36" rot="R90"/>
-<instance part="LED4" gate="G$1" x="91.44" y="76.2" rot="R90"/>
+<instance part="DBG0" gate="G$1" x="91.44" y="106.68" rot="R90"/>
+<instance part="DBG1" gate="G$1" x="91.44" y="96.52" rot="R90"/>
+<instance part="DBG2" gate="G$1" x="91.44" y="86.36" rot="R90"/>
+<instance part="DBG3" gate="G$1" x="91.44" y="76.2" rot="R90"/>
 </instances>
 <busses>
@@
 <wire x1="76.2" y1="109.22" x2="78.74" y2="106.68" width="0.1524" layer="91"/>
 <wire x1="78.74" y1="106.68" x2="88.9" y2="106.68" width="0.1524" layer="91"/>
-<pinref part="LED6" gate="G$1" pin="A"/>
+<pinref part="DBG0" gate="G$1" pin="A"/>
 </segment>
 </net>
@@
 <wire x1="76.2" y1="99.06" x2="78.74" y2="96.52" width="0.1524" layer="91"/>
 <wire x1="78.74" y1="96.52" x2="88.9" y2="96.52" width="0.1524" layer="91"/>
-<pinref part="LED2" gate="G$1" pin="A"/>
+<pinref part="DBG1" gate="G$1" pin="A"/>
 </segment>
 </net>
@@
 <wire x1="76.2" y1="88.9" x2="78.74" y2="86.36" width="0.1524" layer="91"/>
 <wire x1="78.74" y1="86.36" x2="88.9" y2="86.36" width="0.1524" layer="91"/>
-<pinref part="LED3" gate="G$1" pin="A"/>
+<pinref part="DBG2" gate="G$1" pin="A"/>
 </segment>
 </net>
@@
 <wire x1="76.2" y1="78.74" x2="78.74" y2="76.2" width="0.1524" layer="91"/>
 <wire x1="78.74" y1="76.2" x2="88.9" y2="76.2" width="0.1524" layer="91"/>
-<pinref part="LED4" gate="G$1" pin="A"/>
+<pinref part="DBG3" gate="G$1" pin="A"/>
 </segment>
 </net>
@@
 <pinref part="R23" gate="G$1" pin="1"/>
 <wire x1="96.52" y1="76.2" x2="106.68" y2="76.2" width="0.1524" layer="91"/>
-<pinref part="LED4" gate="G$1" pin="C"/>
+<pinref part="DBG3" gate="G$1" pin="C"/>
 </segment>
 </net>
@@
 <pinref part="R22" gate="G$1" pin="1"/>
 <wire x1="106.68" y1="86.36" x2="96.52" y2="86.36" width="0.1524" layer="91"/>
-<pinref part="LED3" gate="G$1" pin="C"/>
+<pinref part="DBG2" gate="G$1" pin="C"/>
 </segment>
 </net>
@@
 <pinref part="R21" gate="G$1" pin="1"/>
 <wire x1="96.52" y1="96.52" x2="106.68" y2="96.52" width="0.1524" layer="91"/>
-<pinref part="LED2" gate="G$1" pin="C"/>
+<pinref part="DBG1" gate="G$1" pin="C"/>
 </segment>
 </net>
@@
 <pinref part="R20" gate="G$1" pin="1"/>
 <wire x1="106.68" y1="106.68" x2="96.52" y2="106.68" width="0.1524" layer="91"/>
-<pinref part="LED6" gate="G$1" pin="C"/>
+<pinref part="DBG0" gate="G$1" pin="C"/>
 </segment>
 </net>
