File: boards/pio/pio.sch (EAGLE design)
At the start: 9 parts

Commit message: Version of PIO to send off for manufacture
Parts:
- added AUDIO: (no value), pinhead:PINHD-1X2
- added C4: 0.1uF, rcl:C-EUC1206
- added H1, H2: MOUNT-HOLE3.2, holes:MOUNT-HOLE3.2
- added IC1: 74AC245DW, 74xx-eu:74AC245DW
- added JOY1_IN, JOY1_OUT, JOY2_IN, JOY2_OUT: (no value), pinhead:PINHD-2X5
- added JP1: (no value), pinhead:PINHD-2X30
- added JP2: (no value), pinhead:PINHD-2X4
Connections:
- removed net N$12: U$1.Y4@19, U$3.P$53
- removed net N$13: U$1.Y3@20, U$3.P$52
- removed net N$14: U$1.Y2@21, U$3.P$51
- removed net N$15: U$1.Y9@14, U$3.P$58
- removed net N$16: U$1.Y8@15, U$3.P$57
- removed net N$17: U$1.Y7@16, U$3.P$56
- removed net N$18: U$1.Y6@17, U$3.P$55
- removed net N$19: U$1.Y5@18, U$3.P$54
- removed net N$2: U$2.AUDIO@E_5, U$3.P$68
- removed net N$20: U$1.Y1@22, U$3.P$50
- removed net N$21: U$1.Y0@23, U$3.P$49
- removed net N$32: U$3.P$48, U$4.Y9@14
- removed net N$33: U$3.P$47, U$4.Y8@15
- removed net N$34: U$3.P$46, U$4.Y7@16
- removed net N$35: U$3.P$45, U$4.Y6@17
- removed net N$36: U$3.P$44, U$4.Y5@18
- removed net N$37: U$3.P$43, U$4.Y4@19
- removed net N$38: U$3.P$42, U$4.Y3@20
- removed net N$39: U$3.P$41, U$4.Y2@21
- removed net N$40: U$3.P$40, U$4.Y1@22
- removed net N$41: U$3.P$39, U$4.Y0@23
- removed net N$50: U$3.P$38, U$5.Y9@14
- removed net N$51: U$3.P$37, U$5.Y8@15
- removed net N$52: U$3.P$36, U$5.Y7@16
- removed net N$53: U$3.P$35, U$5.Y6@17
- removed net N$54: U$3.P$34, U$5.Y5@18
- removed net N$55: U$3.P$33, U$5.Y4@19
- removed net N$56: U$3.P$32, U$5.Y3@20
- removed net N$57: U$3.P$31, U$5.Y2@21
- new net A0: JP1.44, U$1.Y0@23, U$3.P$47
- new net A1: JP1.41, U$3.P$46, U$4.Y9@14
- new net A10: JP1.34, U$3.P$37, U$4.Y0@23
- new net A11: JP1.31, U$3.P$36, U$5.Y9@14
- new net A12: JP1.32, U$3.P$35, U$5.Y8@15
- new net A13: JP1.29, U$3.P$34, U$5.Y7@16
- new net A14: JP1.30, U$3.P$33, U$5.Y6@17
- new net A15: JP1.27, U$3.P$32, U$5.Y5@18
- new net A2: JP1.42, U$3.P$45, U$4.Y8@15
- new net A3: JP1.39, U$3.P$44, U$4.Y7@16
- new net A4: JP1.40, U$3.P$43, U$4.Y6@17
- new net A5: JP1.37, U$3.P$42, U$4.Y5@18
- new net A6: JP1.38, U$3.P$41, U$4.Y4@19
- new net A7: JP1.35, U$3.P$40, U$4.Y3@20
- new net A8: JP1.36, U$3.P$39, U$4.Y2@21
- new net A9: JP1.33, U$3.P$38, U$4.Y1@22
- new net AUDIO: JP1.6, U$2.AUDIO@E_5, U$3.P$66
- new net AUDIO_L: AUDIO.2, JP1.4, U$3.P$67
- new net AUDIO_R: AUDIO.1, JP1.5, U$3.P$68
- new net B02: JP1.47, U$1.Y5@18, U$3.P$52
- new net CCTL: JP1.43, U$1.Y1@22, U$3.P$48
- new net COMMAND: JP2.1, U$3.P$31, U$5.Y4@19
- new net D0: IC1A.A1, JP1.59, U$3.P$64
- new net D1: IC1A.A2, JP1.60, U$3.P$63
- new net D1XX: JP1.50, U$1.Y6@17, U$3.P$53
- new net D2: IC1A.A3, JP1.57, U$3.P$62
- new net D3: IC1A.A4, JP1.58, U$3.P$61
- new net D4: IC1A.A5, JP1.55, U$3.P$60
- new net D5: IC1A.A6, JP1.56, U$3.P$59
- new net D6: IC1A.A7, JP1.53, U$3.P$58
- new net D7: IC1A.A8, JP1.54, U$3.P$57
- new net DATA_OUT: JP2.2, U$3.P$30, U$5.Y3@20
- new net G_IN0: JP1.3
- new net G_IN1: JP1.2
- new net G_IN2: JP1.1
- new net HALT: JP1.52, U$1.Y8@15, U$3.P$55
- new net J1_1: JOY1_IN.1, JOY1_OUT.1, JP1.19, U$3.P$21
- new net J1_2: JOY1_IN.2, JOY1_OUT.2, JP1.20, U$3.P$20
- new net J1_3: JOY1_IN.3, JOY1_OUT.3, JP1.17, U$3.P$19
- new net J1_4: JOY1_IN.5, JOY1_OUT.5, JP1.18, U$3.P$18
- new net J1_5: JOY1_IN.7, JOY1_OUT.7, JP1.15, U$3.P$17
- new net J1_A1: JOY1_IN.8, JOY1_OUT.8, JP1.16, U$3.P$16
- new net J1_A2: JOY1_IN.9, JOY1_OUT.9, JP1.13, U$3.P$15
- new net J2_1: JOY2_IN.1, JOY2_OUT.1, JP1.8, U$3.P$8
- new net J2_2: JOY2_IN.2, JOY2_OUT.2, JP1.7, U$3.P$9
- new net J2_3: JOY2_IN.3, JOY2_OUT.3, JP1.10, U$3.P$10
- new net J2_4: JOY2_IN.5, JOY2_OUT.5, JP1.9, U$3.P$11
- new net J2_5: JOY2_IN.7, JOY2_OUT.7, JP1.12, U$3.P$12
- new net J2_A1: JOY2_IN.8, JOY2_OUT.8, JP1.11, U$3.P$13
- new net J2_A2: JOY2_IN.9, JOY2_OUT.9, JP1.14, U$3.P$14
- new net MTR_CTRL: JP2.3, U$3.P$29, U$5.Y2@21
- new net N$67: IC1A.B8, U$2.D7@C_M
- new net N$68: IC1A.B7, U$2.D6@C_11
- new net N$69: IC1A.B6, U$2.D5@C_7
- new net N$70: IC1A.B5, U$2.D4@C_6
- new net N$71: IC1A.B4, U$2.D3@C_L
- new net N$72: IC1A.B3, U$2.D2@C_8
- new net N$73: IC1A.B2, U$2.D1@C_9
- new net N$74: IC1A.B1, U$2.D0@C_10
- new net REF: JP1.48, U$1.Y4@19, U$3.P$51
- new net RST: JP1.49, U$1.Y7@16, U$3.P$54
- new net RW: JP1.51, U$1.Y9@14, U$3.P$56
- new net S4: JP1.45, U$1.Y3@20, U$3.P$50
- new net S5: JP1.46, U$1.Y2@21, U$3.P$49
- net !EXSEL!: now also JP1.25
- net !IRQ!: now also JP1.28, U$3.P$28; no longer U$3.P$26
- net !MPD!: now also JP1.26, U$3.P$26; no longer U$3.P$28
- net +5V: now also C4.1, IC1P.VCC, JOY1_IN.4, JOY1_OUT.4, JOY2_IN.4, JOY2_OUT.4, JP2.7
- net GND: now also C4.2, IC1A.G, IC1P.GND, JOY1_IN.6, JOY1_OUT.6, JOY2_IN.6, JOY2_OUT.6, U$3.P$65; no longer U$3.P$67
- net RD4: now also JP1.23, U$3.P$25; no longer U$3.P$30
- net RD5: now also JP1.24, U$3.P$24; no longer U$3.P$29
- net SIO_CLK_IN: now also JP1.22, U$3.P$22; no longer U$3.P$25
- net SIO_DATA_IN: now also JP1.21, U$3.P$23; no longer U$3.P$24
Other:
- moved on the sheet: U$3

Commit message: Ok, belay that last. *This* is the one to go to the fab.
Connections:
- net +5V: now also U$6.VCC@1
- net GND: now also U$6.GND@2
- net RW: now also IC1A.DIR
Changed lines of the file:
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@@
 <setting verticaltext="up"/>
 </settings>
-<grid distance="0.1" unitdist="inch" unit="inch" style="lines" multiple="1" display="yes" altdistance="0.01" altunitdist="inch" altunit="inch"/>
+<grid distance="0.1" unitdist="inch" unit="inch" style="lines" multiple="1" display="no" altdistance="0.01" altunitdist="inch" altunit="inch"/>
 <layers>
 <layer number="1" name="Top" color="4" fill="1" visible="no" active="no"/>
@@
 <part name="H1" library="holes" library_urn="urn:adsk.eagle:library:237" deviceset="MOUNT-HOLE" device="3.2" package3d_urn="urn:adsk.eagle:package:14275/1"/>
 <part name="H2" library="holes" library_urn="urn:adsk.eagle:library:237" deviceset="MOUNT-HOLE" device="3.2" package3d_urn="urn:adsk.eagle:package:14275/1"/>
+<part name="SUPPLY15" library="supply2" library_urn="urn:adsk.eagle:library:372" deviceset="GND" device=""/>
+<part name="P+12" library="supply1" library_urn="urn:adsk.eagle:library:371" deviceset="+5V" device=""/>
 </parts>
 <sheets>
@@
 <instance part="H1" gate="G$1" x="309.88" y="-17.78"/>
 <instance part="H2" gate="G$1" x="309.88" y="-22.86"/>
+<instance part="SUPPLY15" gate="GND" x="-53.34" y="111.76"/>
+<instance part="P+12" gate="1" x="-53.34" y="144.78"/>
 </instances>
 <busses>
@@
 <wire x1="163.83" y1="134.62" x2="163.83" y2="121.92" width="0.1524" layer="91"/>
 </segment>
+<segment>
+<pinref part="U$6" gate="G$1" pin="GND@2"/>
+<pinref part="SUPPLY15" gate="GND" pin="GND"/>
+<wire x1="-48.26" y1="116.84" x2="-53.34" y2="116.84" width="0.1524" layer="91"/>
+<wire x1="-53.34" y1="116.84" x2="-53.34" y2="114.3" width="0.1524" layer="91"/>
+</segment>
 </net>
 <net name="AUDIO" class="0">
@@
 <wire x1="261.62" y1="25.4" x2="261.62" y2="43.18" width="0.1524" layer="91"/>
 </segment>
+<segment>
+<pinref part="U$6" gate="G$1" pin="VCC@1"/>
+<pinref part="P+12" gate="1" pin="+5V"/>
+<wire x1="-48.26" y1="137.16" x2="-53.34" y2="137.16" width="0.1524" layer="91"/>
+<wire x1="-53.34" y1="137.16" x2="-53.34" y2="142.24" width="0.1524" layer="91"/>
+</segment>
 </net>
 <net name="N$22" class="0">
@@
 <wire x1="114.3" y1="5.08" x2="111.76" y2="7.62" width="0.1524" layer="91"/>
 <pinref part="U$1" gate="G$1" pin="Y9@14"/>
-<wire x1="111.76" y1="7.62" x2="99.06" y2="7.62" width="0.1524" layer="91"/>
+<wire x1="111.76" y1="7.62" x2="104.14" y2="7.62" width="0.1524" layer="91"/>
 <label x="111.252" y="7.366" size="1.778" layer="95" rot="R180"/>
-</segment>
-<segment>
+<pinref part="IC1" gate="A" pin="DIR"/>
+<wire x1="104.14" y1="7.62" x2="99.06" y2="7.62" width="0.1524" layer="91"/>
+<wire x1="91.44" y1="-22.86" x2="104.14" y2="-22.86" width="0.1524" layer="91"/>
+<wire x1="104.14" y1="-22.86" x2="104.14" y2="7.62" width="0.1524" layer="91"/>
+<junction x="104.14" y="7.62"/>
+</segment>
+<segment>
