File: boards/xio/xio.sch (EAGLE design)
At the start: 1 part

Commit message: Checkpoint
Connections:
- new net VDD: U$1G$1.VDD@C19, U$1G$1.VDD@C3, U$1G$1.VDD@E13, U$1G$1.VDD@E14, U$1G$1.VDD@E17, U$1G$1.VDD@E18, U$1G$1.VDD@E4, U$1G$1.VDD@E5, U$1G$1.VDD@E8, U$1G$1.VDD@E9, U$1G$1.VDD@F12, U$1G$1.VDD@F13, U$1G$1.VDD@F14, U$1G$1.VDD@F15, U$1G$1.VDD@F16, U$1G$1.VDD@F17, U$1G$1.VDD@F18, U$1G$1.VDD@F4, U$1G$1.VDD@F5, U$1G$1.VDD@F6, U$1G$1.VDD@F7, U$1G$1.VDD@F8, U$1G$1.VDD@F9, U$1G$1.VDD@H19, U$1G$1.VDD@H3, U$1G$1.VDD@J19, U$1G$1.VDD@J3, U$1G$1.VDD@N19, U$1G$1.VDD@N3, U$1G$1.VDD@P19, U$1G$1.VDD@P3, U$1G$1.VDD@T10, U$1G$1.VDD@T12, U$1G$1.VDD@T13, U$1G$1.VDD@T14, U$1G$1.VDD@T16, U$1G$1.VDD@T17, U$1G$1.VDD@T18, U$1G$1.VDD@T4, U$1G$1.VDD@T5, U$1G$1.VDD@T6, U$1G$1.VDD@T8, U$1G$1.VDD@T9, U$1G$1.VDD@U13, U$1G$1.VDD@U14, U$1G$1.VDD@U17, U$1G$1.VDD@U18, U$1G$1.VDD@U4, U$1G$1.VDD@U5, U$1G$1.VDD@U9
- new net VDDIO: U$1G$1.OTP_VCC@C11, U$1G$1.VDDIO@A11, U$1G$1.VDDIO@A2, U$1G$1.VDDIO@A20, U$1G$1.VDDIO@AA11, U$1G$1.VDDIO@AA2, U$1G$1.VDDIO@AA20, U$1G$1.VDDIO@D7, U$1G$1.VDDIO@E15, U$1G$1.VDDIO@E7, U$1G$1.VDDIO@F2, U$1G$1.VDDIO@F20, U$1G$1.VDDIO@L1, U$1G$1.VDDIO@L21, U$1G$1.VDDIO@T2, U$1G$1.VDDIO@T20, U$1G$1.VDDIO@U11, U$1G$1.VDDIO@U15, U$1G$1.VDDIO@U7, U$1G$1.VDDIO_T@A16, U$1G$1.VDDIO_T@A6

Commit message: Progress checkpoint
Parts:
- added C1, C10, C11, C12, C13, C14, C15, C16, C17, C18, C19, C2, C20, C21, C22, C23, C24, C25, C26, C27, C28, C29, C3, C30, C31, C32, C33, C4, C5, C6, C7, C8, C9: 0.1uF, rcl:C-EUC0402K
- added C34, C35: 10uF, rcl:C-EUC0402K
- added R1: 2.2R, rcl:R-EU_R0402
- added R2: 0, rcl:R-EU_R0402
Connections:
- new net N$1: C1.1, R1.1, U$1G$1.PLL_AVDD@F11
- new net N$2: C1.2, R2.2, U$1G$1.PLL_AGND@F10
- net GND: now also C10.2, C11.2, C12.2, C13.2, C14.2, C15.2, C16.2, C17.2, C18.2, C19.2, C2.2, C20.2, C21.2, C22.2, C23.2, C24.2, C25.2, C26.2, C27.2, C28.2, C29.2, C3.2, C30.2, C31.2, C32.2, C33.2, C34.2, C35.2, C4.2, C5.2, C6.2, C7.2, C8.2, C9.2, R2.1
- net VDD: now also C18.1, C19.1, C20.1, C21.1, C22.1, C23.1, C24.1, C25.1, C26.1, C27.1, C28.1, C29.1, C30.1, C31.1, C32.1, C33.1, C35.1, R1.2
- net VDDIO: now also C10.1, C11.1, C12.1, C13.1, C14.1, C15.1, C16.1, C17.1, C2.1, C3.1, C34.1, C4.1, C5.1, C6.1, C7.1, C8.1, C9.1
Other:
- note added: "Vdd should supply 1.4A - AP7363-10D-13 : fixed, 1vout, 5.5vin, 1.5A , 2x10uF cap - AP7363-33D-13 : fixed, 3.3vout, 5.5vin, 1.5A, 2x 10uF cap"
- note removed: "Vdd should supply 1.4A"

Commit message: Start to realise that this board is going to be big…
Parts:
- removed C11, C12, C13, C14, C15, C16, C17, C30, C31, C32, C33: 0.1uF, rcl:C-EUC0402K
- removed R2: 0, rcl:R-EU_R0402
- added X1, X2, X3, X4, X5, X6, X7: PCI-E-164SOCKET, con-pc:PCI-E-164SOCKET
- R1: value 2.2R -> 4.7R
- U$1: value XEF-232-1024-FB374 -> XEF-216-512-FB236; device sjg-xmos:XEF-232-1024-FB374 -> sjg-xmos:XEF-216-512-FB236
Connections:
- removed net N$2: C1.2, R2.2, U$1G$1.PLL_AGND@F10
- removed net VDDIO: C10.1, C11.1, C12.1, C13.1, C14.1, C15.1, C16.1, C17.1, C2.1, C3.1, C34.1, C4.1, C5.1, C6.1, C7.1, C8.1, C9.1, U$1G$1.OTP_VCC@C11, U$1G$1.VDDIO@A11, U$1G$1.VDDIO@A2, U$1G$1.VDDIO@A20, U$1G$1.VDDIO@AA11, U$1G$1.VDDIO@AA2, U$1G$1.VDDIO@AA20, U$1G$1.VDDIO@D7, U$1G$1.VDDIO@E15, U$1G$1.VDDIO@E7, U$1G$1.VDDIO@F2, U$1G$1.VDDIO@F20, U$1G$1.VDDIO@L1, U$1G$1.VDDIO@L21, U$1G$1.VDDIO@T2, U$1G$1.VDDIO@T20, U$1G$1.VDDIO@U11, U$1G$1.VDDIO@U15, U$1G$1.VDDIO@U7, U$1G$1.VDDIO_T@A16, U$1G$1.VDDIO_T@A6
- new net +3V3: U$1G$1.OTP_VCC@A12, U$1G$1.OTP_VCC@B12, U$1G$1.VDDIOL@A2, U$1G$1.VDDIOL@A3, U$1G$1.VDDIOL@B2, U$1G$1.VDDIOL@B3, U$1G$1.VDDIOL@C3, U$1G$1.VDDIOL@V2, U$1G$1.VDDIOL@V3, U$1G$1.VDDIOL@W2, U$1G$1.VDDIOR@A18, U$1G$1.VDDIOR@B18, U$1G$1.VDDIOR@B19, U$1G$1.VDDIOR@V17, U$1G$1.VDDIOR@V18, U$1G$1.VDDIOR@W17, U$1G$1.VDDIOR@W18, U$1G$1.VDDIOT@F10
- new net 3V3: C10.1, C2.1, C3.1, C34.1, C4.1, C5.1, C6.1, C7.1, C8.1, C9.1
- net GND: now also C1.2, U$1G$1.GND@A19, U$1G$1.GND@G10, U$1G$1.GND@G12, U$1G$1.GND@G8, U$1G$1.GND@H10, U$1G$1.GND@H11, U$1G$1.GND@H12, U$1G$1.GND@H13, U$1G$1.GND@H7, U$1G$1.GND@H8, U$1G$1.GND@H9, U$1G$1.GND@J10, U$1G$1.GND@J12, U$1G$1.GND@K10, U$1G$1.GND@K11, U$1G$1.GND@K12, U$1G$1.GND@L10, U$1G$1.GND@L12, U$1G$1.GND@M10, U$1G$1.GND@M11, U$1G$1.GND@M12, U$1G$1.GND@N10, U$1G$1.GND@N12, U$1G$1.GND@W1, U$1G$1.GND@W19, U$1G$1.PLL_AGND@F14; no longer C11.2, C12.2, C13.2, C14.2, C15.2, C16.2, C17.2, C30.2, C31.2, C32.2, C33.2, R2.1, U$1G$1.GND@A21, U$1G$1.GND@AA1, U$1G$1.GND@AA21, U$1G$1.GND@B11, U$1G$1.GND@C15, U$1G$1.GND@C7, U$1G$1.GND@D6, U$1G$1.GND@E16, U$1G$1.GND@E6, U$1G$1.GND@F19, U$1G$1.GND@F3, U$1G$1.GND@J13, U$1G$1.GND@J14, U$1G$1.GND@J15, U$1G$1.GND@J16, U$1G$1.GND@J17, U$1G$1.GND@J5, U$1G$1.GND@J6, U$1G$1.GND@J7, U$1G$1.GND@J9, U$1G$1.GND@K14, U$1G$1.GND@K15, U$1G$1.GND@K16, U$1G$1.GND@K17, U$1G$1.GND@K5, U$1G$1.GND@K6, U$1G$1.GND@L13, U$1G$1.GND@L14, U$1G$1.GND@L15, U$1G$1.GND@L16, U$1G$1.GND@L17, U$1G$1.GND@L2, U$1G$1.GND@L20, U$1G$1.GND@L5, U$1G$1.GND@L6, U$1G$1.GND@L7, U$1G$1.GND@L9, U$1G$1.GND@M14, U$1G$1.GND@M15, U$1G$1.GND@M16, U$1G$1.GND@M17, U$1G$1.GND@M5, U$1G$1.GND@M6, U$1G$1.GND@N13, U$1G$1.GND@N14, U$1G$1.GND@N15, U$1G$1.GND@N16, U$1G$1.GND@N17, U$1G$1.GND@N5, U$1G$1.GND@N6, U$1G$1.GND@N7, U$1G$1.GND@N9, U$1G$1.GND@T11, U$1G$1.GND@T19, U$1G$1.GND@T3, U$1G$1.GND@U16, U$1G$1.GND@U6, U$1G$1.GND@W15, U$1G$1.GND@W7, U$1G$1.GND@Y11
- net N$1: now also U$1G$1.PLL_AVDD@F13; no longer U$1G$1.PLL_AVDD@F11
- net VDD: now also U$1G$1.VDD@F11, U$1G$1.VDD@G14, U$1G$1.VDD@G6, U$1G$1.VDD@H14, U$1G$1.VDD@H6, U$1G$1.VDD@J14, U$1G$1.VDD@J6, U$1G$1.VDD@K14, U$1G$1.VDD@K6, U$1G$1.VDD@L14, U$1G$1.VDD@L6, U$1G$1.VDD@M14, U$1G$1.VDD@M6, U$1G$1.VDD@N14, U$1G$1.VDD@N6, U$1G$1.VDD@P11, U$1G$1.VDD@P12, U$1G$1.VDD@P13, U$1G$1.VDD@P6, U$1G$1.VDD@P7, U$1G$1.VDD@P8; no longer C30.1, C31.1, C32.1, C33.1, U$1G$1.VDD@C19, U$1G$1.VDD@C3, U$1G$1.VDD@E13, U$1G$1.VDD@E14, U$1G$1.VDD@E17, U$1G$1.VDD@E18, U$1G$1.VDD@E4, U$1G$1.VDD@E5, U$1G$1.VDD@E8, U$1G$1.VDD@E9, U$1G$1.VDD@F13, U$1G$1.VDD@F14, U$1G$1.VDD@F15, U$1G$1.VDD@F16, U$1G$1.VDD@F17, U$1G$1.VDD@F18, U$1G$1.VDD@F4, U$1G$1.VDD@F5, U$1G$1.VDD@F6, U$1G$1.VDD@F7, U$1G$1.VDD@H19, U$1G$1.VDD@H3, U$1G$1.VDD@J19, U$1G$1.VDD@J3, U$1G$1.VDD@N19, U$1G$1.VDD@N3, U$1G$1.VDD@P19, U$1G$1.VDD@P3, U$1G$1.VDD@T10, U$1G$1.VDD@T12, U$1G$1.VDD@T13, U$1G$1.VDD@T14, U$1G$1.VDD@T16, U$1G$1.VDD@T17, U$1G$1.VDD@T18, U$1G$1.VDD@T4, U$1G$1.VDD@T5, U$1G$1.VDD@T6, U$1G$1.VDD@T8, U$1G$1.VDD@T9, U$1G$1.VDD@U13, U$1G$1.VDD@U14, U$1G$1.VDD@U17, U$1G$1.VDD@U18, U$1G$1.VDD@U4, U$1G$1.VDD@U5, U$1G$1.VDD@U9
Other:
- note removed: "KSZ9031MNX works well, handles 3.3v"

Commit message: Board checkpoint
Parts:
- added C11, C12, C14: 10uF, rcl:C-EUC0402K
- added C13, C15: 1uF, rcl:C-EUC0402K
- added C16: 120pF, rcl:C-EUC0402
- added C17: 0.1uF, rcl:C-EUC0402
- added H1, H2, H3, H4, H5: MOUNT-HOLE3.2, holes:MOUNT-HOLE3.2
- added R27: 47K, rcl:R-EU_R0402
- added U$2: AP7363-330-13, sjg-power:AP7363
- added U$3: LD49150, sjg-power:LD49150
- added U$6: TPS3808G33DBVR, sjg-power:TPS3808G33DBVR
Connections:
- new net +5V: C11.1, C13.1, C15.1, U$2.IN@1, U$3.VBIAS, U$3.VIN
- new net EN_1V0: R27.1, U$3.EN, U$6.!RESET!@1
- new net N$13: C16.1, U$6.CT@4
- net +3V3: now also C12.1, C17.1, R27.2, U$2.OUT@3, U$6.SENSE@5, U$6.VCC@6
- net GND: now also C11.2, C12.2, C13.2, C14.2, C15.2, C16.2, C17.2, U$2.GND@2, U$3.GND, U$6.GND@2
- net VDD: now also C14.1, U$3.VOUT
Other:
- note added: "Duplicate per slot"
- note added: "t(Delay) = 1.2ms"

Commit message: Route power to the slots
Parts:
- removed R27: 47K, rcl:R-EU_R0402
- added C30: 10nF, rcl:C-EUC0402
- added C31, C33, C36: 0.1uF, rcl:C-EUC0402
- added C32: 120pF, rcl:C-EUC0402
- added C37, C38, C39, C40, C41, C42, C43, C44, C45, C46, C47, C48, C49, C50: 10uF, rcl:C-EUC0402K
- added JTAG5V1: PSU, pinhead:PINHD-1X2
- added PJ-102AH: PJ-102AH, adafruit:2.1MMJACKTHM
- added R2: 1K, rcl:R-EU_R0402
- added R3: 47K, rcl:R-EU_R0402
- added R4, R5: 47k, rcl:R-EU_R0402
- added RESET_SW: (no value), SparkFun:TAC_SWITCHPTH
- added U$10, U$11, U$12, U$13, U$7, U$8, U$9: AP7363-330-13, sjg-power:AP7363
- added U$4: TPS3808G33DBVR, sjg-power:TPS3808DBVR
- added U$5: 74LVC1G07SE-7, sjg-logic:74LVC1G07SE-7
- added U1: 24 MHz Osc. (F535L-24), SparkFun:OSCILLATOR5X3-PIN1-INDICATED
- added XTAG1: 1175-1618-ND, pinhead:PINHD-2X10/90
- C16: value 120pF -> 0.1uF
- C17: value 0.1uF -> 120pF
- U$6: value TPS3808G33DBVR -> TPS3808G09DBVR; device sjg-power:TPS3808G33DBVR -> sjg-power:TPS3808DBVR
Connections:
- removed net EN_1V0: R27.1, U$3.EN, U$6.!RESET!@1
- removed net N$13: C16.1, U$6.CT@4
- new net !RESET!: R5.1, U$1G$2.!RST!@C6, U$1G$2.!TRST!@B6, U$5.Y@4, U$6.!RESET!@1
- new net JTAG_DN0: XTAG1.14
- new net JTAG_DN1: XTAG1.18
- new net JTAG_UP0: XTAG1.10
- new net JTAG_UP1: XTAG1.6
- new net N$10: C36.1, RESET_SW.1, RESET_SW.2, U$6.!MR!@3
- new net N$2: R2.1
- new net N$3: U$1G$2.CLK@A6, U1.OUT
- new net N$4: C31.2, R3.1, U$3.EN, U$4.VDD@6
- new net N$5: C32.1, U$4.CT@4
- new net N$7: R4.1, U$5.A@2, XTAG1.15
- new net N$8: JTAG5V1.2, XTAG1.1
- new net N$9: C17.2, U$6.CT@4
- new net S1_V33: C38.1, U$7.OUT@3, X1.A5, X1.A6, X1.B5, X1.B6
- new net S2_V33: C40.1, U$8.OUT@3, X2.A5, X2.A6, X2.B5, X2.B6
- new net S3_V33: C42.1, U$9.OUT@3, X3.A5, X3.A6, X3.B5, X3.B6
- new net S4_V33: C44.1, U$10.OUT@3, X4.A5, X4.A6, X4.B5, X4.B6
- new net S5_V33: C46.1, U$11.OUT@3, X5.A5, X5.A6, X5.B5, X5.B6
- new net S6_V33: C48.1, U$12.OUT@3, X6.A5, X6.A6, X6.B5, X6.B6
- new net S7_V33: C50.1, U$13.OUT@3, X7.A5, X7.A6, X7.B5, X7.B6
- new net TCK: U$1G$2.TCK@A5, XTAG1.9
- new net TDI: U$1G$2.TDI@C4, XTAG1.5
- new net TDO: U$1G$2.TDO@B4, XTAG1.13
- new net TMS: U$1G$2.TMS@B5, XTAG1.7
- new net UART_RX: XTAG1.19
- new net UART_TX: XTAG1.17
- new net VCCIO: C31.1, R3.2
- net +3V3: now also C16.1, C30.2, C33.1, R2.2, R4.2, R5.2, U$4.SENSE@5, U$5.VCC@5, U$6.VDD@6, U1.VCC; no longer C17.1, R27.2, U$6.SENSE@5, U$6.VCC@6
- net +5V: now also C37.1, C39.1, C41.1, C43.1, C45.1, C47.1, C49.1, JTAG5V1.1, PJ-102AH.TIP, U$10.IN@1, U$11.IN@1, U$12.IN@1, U$13.IN@1, U$7.IN@1, U$8.IN@1, U$9.IN@1, X1.A1, X1.A2, X1.B1, X1.B2, X2.A1, X2.A2, X2.B1, X2.B2, X3.A1, X3.A2, X3.B1, X3.B2, X4.A1, X4.A2, X4.B1, X4.B2, X5.A1, X5.A2, X5.B1, X5.B2, X6.A1, X6.A2, X6.B1, X6.B2, X7.A1, X7.A2, X7.B1, X7.B2
- net GND: now also C17.1, C30.1, C32.2, C33.2, C36.2, C37.2, C38.2, C39.2, C40.2, C41.2, C42.2, C43.2, C44.2, C45.2, C46.2, C47.2, C48.2, C49.2, C50.2, PJ-102AH.RING, RESET_SW.3, RESET_SW.4, U$10.GND@2, U$11.GND@2, U$12.GND@2, U$13.GND@2, U$4.GND@2, U$5.GND@3, U$7.GND@2, U$8.GND@2, U$9.GND@2, U1.GND, X1.A3, X1.A4, X1.B3, X1.B4, X2.A3, X2.A4, X2.B3, X2.B4, X3.A3, X3.A4, X3.B3, X3.B4, X4.A3, X4.A4, X4.B3, X4.B4, X5.A3, X5.A4, X5.B3, X5.B4, X6.A3, X6.A4, X6.B3, X6.B4, X7.A3, X7.A4, X7.B3, X7.B4, XTAG1.12, XTAG1.16, XTAG1.20, XTAG1.4, XTAG1.8; no longer C17.2
- net VDD: now also U$6.SENSE@5
Other:
- note added: "3.3v from +5v"
- note added: "CLOCK"
- note added: "Clock is 24 MHz (within PLL range)"
- note added: "Gated 1v from +5v"
- note added: "Intentionally left unconnected"
- note added: "Mate with jyh05010000b"
- note added: "Mode0 and Mode1 left unconnected. At 24MHz, with pull-ups to 2'b11, will boot at 384 MHz !DEBUG! not needed for single CPU"
- note added: "Monitor the VDD line and reset if it falls below 0.9v. In addition, allow a manual reset of the chip via button"
- note added: "Power entry"
- note added: "RESET"
- note added: "SLOTS 1,2,3"
- note added: "SLOTS 4,5,6,7"
- note added: "Slot 1 power"
- note added: "Slot 2 power"
- note added: "Slot 3 power"
- note added: "Slot 4 power"
- note added: "Slot 5 power"
- note added: "Slot 7 power"
- note added: "XMOS CLK, XTAG, RESET"
- note added: "XMOS PORT X0"
- note added: "XMOS PORT X1"
- note added: "XMOS POWER"
- note added: "XMOS USB"
- note added: "XTAG"

Commit message: Start to route the expansion bus
Parts:
- added U$14: HE11-RDA-101-4, sjg-vhdci:HE11-RDA-101-4
Connections:
- new net VHDCI_A00: U$14.P$47, X1.A15, X2.A15, X3.A15, X4.A15, X5.A15, X6.A15, X7.A15
- new net VHDCI_A01: U$14.P$46, X1.A16, X2.A16, X3.A16, X4.A16, X5.A16, X6.A16, X7.A16
- new net VHDCI_A02: U$14.P$45, X1.A17, X2.A17, X3.A17, X4.A17, X5.A17, X6.A17, X7.A17
- new net VHDCI_A03: U$14.P$44, X1.A18, X2.A18, X3.A18, X4.A18, X5.A18, X6.A18, X7.A18
- new net VHDCI_A04: U$14.P$43, X1.A19, X2.A19, X3.A19, X4.A19, X5.A19, X6.A19, X7.A19
- new net VHDCI_A05: U$14.P$42, X1.A20, X2.A20, X3.A20, X4.A20, X5.A20, X6.A20, X7.A20
- new net VHDCI_A06: U$14.P$41, X1.A21, X2.A21, X3.A21, X4.A21, X5.A21, X6.A21, X7.A21
- new net VHDCI_A07: U$14.P$40, X1.A22, X2.A22, X3.A22, X4.A22, X5.A22, X6.A22, X7.A22
- new net VHDCI_A08: U$14.P$39, X1.A23, X2.A23, X3.A23, X4.A23, X5.A23, X6.A23, X7.A23
- new net VHDCI_A09: U$14.P$38, X1.A24, X2.A24, X3.A24, X4.A24, X5.A24, X6.A24, X7.A24
- new net VHDCI_A10: U$14.P$37, X1.A25, X2.A25, X3.A25, X4.A25, X5.A25, X6.A25, X7.A25
- new net VHDCI_A11: U$14.P$36, X1.A26, X2.A26, X3.A26, X4.A26, X5.A26, X6.A26, X7.A26
- new net VHDCI_A12: U$14.P$35, X1.A27, X2.A27, X3.A27, X4.A27, X5.A27, X6.A27, X7.A27
- new net VHDCI_A13: U$14.P$34, X1.A28, X2.A28, X3.A28, X4.A28, X5.A28, X6.A28, X7.A28
- new net VHDCI_A14: U$14.P$33, X1.A29, X2.A29, X3.A29, X4.A29, X5.A29, X6.A29, X7.A29
- new net VHDCI_A15: U$14.P$32, X1.A30, X2.A30, X3.A30, X4.A30, X5.A30, X6.A30, X7.A30
- new net VHDCI_AUDIO: U$14.P$66, X1.A31, X2.A31, X3.A31, X4.A31, X5.A31, X6.A31, X7.A31
- new net VHDCI_AUDIO_L: U$14.P$67, X1.A32, X2.A32, X3.A32, X4.A32, X5.A32, X6.A32, X7.A32
- new net VHDCI_AUDIO_R: U$14.P$68, X1.A33, X2.A33, X3.A33, X4.A33, X5.A33, X6.A33, X7.A33
- new net VHDCI_CCTL: U$14.P$48, X1.A34, X2.A34, X3.A34, X4.A34, X5.A34, X6.A34, X7.A34
- new net VHDCI_CLK: U$14.P$52, X1.A35, X2.A35, X3.A35, X4.A35, X5.A35, X6.A35, X7.A35
- new net VHDCI_COMMAND: U$14.P$31, X1.A36, X2.A36, X3.A36, X4.A36, X5.A36, X6.A36, X7.A36
- new net VHDCI_D00: U$14.P$64, X1.A37, X2.A37, X3.A37, X4.A37, X5.A37, X6.A37, X7.A37
- new net VHDCI_D01: U$14.P$63, X1.A38, X2.A38, X3.A38, X4.A38, X5.A38, X6.A38, X7.A38
- new net VHDCI_D02: U$14.P$62, X1.A39, X2.A39, X3.A39, X4.A39, X5.A39, X6.A39, X7.A39
- new net VHDCI_D03: U$14.P$61, X1.A40, X2.A40, X3.A40, X4.A40, X5.A40, X6.A40, X7.A40
- new net VHDCI_D04: U$14.P$60, X1.A41, X2.A41, X3.A41, X4.A41, X5.A41, X6.A41, X7.A41
- new net VHDCI_D05: U$14.P$59, X1.A42, X2.A42, X3.A42, X4.A42, X5.A42, X6.A42, X7.A42
- new net VHDCI_D06: U$14.P$58, X1.A43, X2.A43, X3.A43, X4.A43, X5.A43, X6.A43, X7.A43
- new net VHDCI_D07: U$14.P$57, X1.A44, X2.A44, X3.A44, X4.A44, X5.A44, X6.A44, X7.A44
- new net VHDCI_D1XX: U$14.P$53, X1.A45, X2.A45, X3.A45, X4.A45, X5.A45, X6.A45, X7.A45
- new net VHDCI_DATA_OUT: U$14.P$30, X1.A46, X2.A46, X3.A46, X4.A46, X5.A46, X6.A46, X7.A46
- new net VHDCI_EXSEL: U$14.P$27, X1.A47, X2.A47, X3.A47, X4.A47, X5.A47, X6.A47, X7.A47
- new net VHDCI_GND: U$14.P$65, X1.A48, X2.A48, X3.A48, X4.A48, X5.A48, X6.A48, X7.A48
- new net VHDCI_HALT: U$14.P$55, X1.A49, X2.A49, X3.A49, X4.A49, X5.A49, X6.A49, X7.A49
- new net VHDCI_IRQ: U$14.P$28, X1.A50, X2.A50, X3.A50, X4.A50, X5.A50, X6.A50, X7.A50
- new net VHDCI_J1_1: U$14.P$21, X1.A51, X2.A51, X3.A51, X4.A51, X5.A51, X6.A51, X7.A51
- new net VHDCI_J1_2: U$14.P$20, X1.A52, X2.A52, X3.A52, X4.A52, X5.A52, X6.A52, X7.A52
- new net VHDCI_J1_3: U$14.P$19, X1.A53, X2.A53, X3.A53, X4.A53, X5.A53, X6.A53, X7.A53
- new net VHDCI_J1_4: U$14.P$18, X1.A54, X2.A54, X3.A54, X4.A54, X5.A54, X6.A54, X7.A54
- new net VHDCI_J1_5: U$14.P$17, X1.A55, X2.A55, X3.A55, X4.A55, X5.A55, X6.A55, X7.A55
- new net VHDCI_J1_A1: U$14.P$16, X1.A56, X2.A56, X3.A56, X4.A56, X5.A56, X6.A56, X7.A56
- new net VHDCI_J1_A2: X1.A57, X2.A57, X3.A57, X4.A57, X5.A57, X6.A57, X7.A57
- new net VHDCI_J2_1: U$14.P$8, X1.A58, X2.A58, X3.A58, X4.A58, X5.A58, X6.A58, X7.A58
- new net VHDCI_J2_2: U$14.P$9, X1.A59, X2.A59, X3.A59, X4.A59, X5.A59, X6.A59, X7.A59
- new net VHDCI_J2_3: U$14.P$10, X1.A60, X2.A60, X3.A60, X4.A60, X5.A60, X6.A60, X7.A60
- new net VHDCI_J2_4: U$14.P$11, X1.A61, X2.A61, X3.A61, X4.A61, X5.A61, X6.A61, X7.A61
- new net VHDCI_J2_5: U$14.P$12, X1.A62, X2.A62, X3.A62, X4.A62, X5.A62, X6.A62, X7.A62
- new net VHDCI_J2_A1: U$14.P$13, X1.A63, X2.A63, X3.A63, X4.A63, X5.A63, X6.A63, X7.A63
- new net VHDCI_J2_A2: U$14.P$14, U$14.P$15, X1.A64, X2.A64, X3.A64, X4.A64, X5.A64, X6.A64, X7.A64
- new net VHDCI_MPD: U$14.P$26, X1.A65, X2.A65, X3.A65, X4.A65, X5.A65, X6.A65, X7.A65
- new net VHDCI_MTR_CTRL: U$14.P$29, X1.A66, X2.A66, X3.A66, X4.A66, X5.A66, X6.A66, X7.A66
- new net VHDCI_NC1: U$14.P$1, X1.A67, X2.A67, X3.A67, X4.A67, X5.A67, X6.A67, X7.A67
- new net VHDCI_NC2: U$14.P$2, X1.A68, X2.A68, X3.A68, X4.A68, X5.A68, X6.A68, X7.A68
- new net VHDCI_NC3: U$14.P$3, X1.A69, X2.A69, X3.A69, X4.A69, X5.A69, X6.A69, X7.A69
- new net VHDCI_NC4: U$14.P$4, X1.A70, X2.A70, X3.A70, X4.A70, X5.A70, X6.A70, X7.A70
- new net VHDCI_NC5: U$14.P$5, X1.A71, X2.A71, X3.A71, X4.A71, X5.A71, X6.A71, X7.A71
- new net VHDCI_NC6: U$14.P$6, X1.A72, X2.A72, X3.A72, X4.A72, X5.A72, X6.A72, X7.A72
- new net VHDCI_NC7: U$14.P$7, X1.A73, X2.A73, X3.A73, X4.A73, X5.A73, X6.A73, X7.A73
- new net VHDCI_RD4: U$14.P$25, X1.A74, X2.A74, X3.A74, X4.A74, X5.A74, X6.A74, X7.A74
- new net VHDCI_RD5: U$14.P$24, X1.A75, X2.A75, X3.A75, X4.A75, X5.A75, X6.A75, X7.A75
- new net VHDCI_REF: U$14.P$51, X1.A76, X2.A76, X3.A76, X4.A76, X5.A76, X6.A76, X7.A76
- new net VHDCI_RST: U$14.P$54, X1.A77, X2.A77, X3.A77, X4.A77, X5.A77, X6.A77, X7.A77
- new net VHDCI_RW: U$14.P$56, X1.A78, X2.A78, X3.A78, X4.A78, X5.A78, X6.A78, X7.A78
- new net VHDCI_S4: U$14.P$50, X1.A79, X2.A79, X3.A79, X4.A79, X5.A79, X6.A79, X7.A79
- new net VHDCI_S5: U$14.P$49, X1.A80, X2.A80, X3.A80, X4.A80, X5.A80, X6.A80, X7.A80
- new net VHDCI_SIO_CLK_IN: U$14.P$22, X1.A81, X2.A81, X3.A81, X4.A81, X5.A81, X6.A81, X7.A81
- new net VHDCI_SIO_DATA_IN: U$14.P$23, X1.A82, X2.A82, X3.A82, X4.A82, X5.A82, X6.A82, X7.A82
- net GND: now also U$14.P$69, U$14.P$70, U$14.P$71, U$14.P$72
Other:
- note added: "SLOT POWER"
- note added: "USB not used in this design"
- note added: "VHDCI"
- note added: "VHDCI signals"
- note removed: "Duplicate per slot"
- note removed: "See page 27 for USB routing"

Commit message: Add in the architecture selector
Parts:
- added ARCH_ID: 209-4MS, special:SW_DIP-4
- added R6, R7, R8, R9: 47k, rcl:R-EU_R0402
Connections:
- new net ARCH0: ARCH_ID.1, R9.1, X1.B7, X2.B7, X3.B7, X4.B7, X5.B7, X6.B7, X7.B7
- new net ARCH1: ARCH_ID.2, R8.1, X1.B8, X2.B8, X3.B8, X4.B8, X5.B8, X6.B8, X7.B8
- new net ARCH2: ARCH_ID.3, R7.1, X1.B9, X2.B9, X3.B9, X4.B9, X5.B9, X6.B9, X7.B9
- new net ARCH3: ARCH_ID.4, R6.1, X1.B10, X2.B10, X3.B10, X4.B10, X5.B10, X6.B10, X7.B10
- net +3V3: now also ARCH_ID.5, ARCH_ID.6, ARCH_ID.7, ARCH_ID.8
- net GND: now also R6.2, R7.2, R8.2, R9.2, X1.A8, X1.A9, X2.A7, X2.A9, X3.A9, X4.A7, X4.A8, X5.A8, X6.A7
- net S1_V33: now also X1.A7
- net S2_V33: now also X2.A8
- net S3_V33: now also X3.A7, X3.A8
- net S4_V33: now also X4.A9
- net S5_V33: now also X5.A7, X5.A9
- net S6_V33: now also X6.A8, X6.A9
- net S7_V33: now also X7.A7, X7.A8, X7.A9
Other:
- note added: "Architecture Selection"
- note added: "VHDCI, ARCH"
- note removed: "VHDCI"
