File: boards/xio/xio.sch (EAGLE design)
At the start: 294 parts, among them CN3 J00-0065NL, U2 LAN8742A-CZ, X2 USB-A, Y1 NX3225SA-12.000MHZ-STD-CSR-1, Y2 NX3225SA-12.000MHZ-STD-CSR-1, Y3 NX3225SA-25.000MHZ-STD-CSR-1

Commit message: More updates for the ‘H’ XIO part
Parts:
- removed C19, C20: 0.1uF, rcl:C-EUC0402K
- removed C52: 4.7uF, rcl:C-EUC0402K
- removed PSRAM: IS66WV51216EBLL, sjg-ram:IS66WV51216EBLL
- added SDRAM1: IS42S32800J, sjg-sdram:IS42S32800J
Connections:
- removed net XIO_RAM_!CS!: PSRAM.!CS1!@6
- removed net XIO_RAM_!LB!: PSRAM.!LB!@39
- removed net XIO_RAM_!OE!: PSRAM.!OE!@41
- removed net XIO_RAM_!UB!: PSRAM.!UB!@40
- removed net XIO_RAM_!WE!: PSRAM.!WE!@17
- removed net XIO_RAM_A0: PSRAM.A0@5
- removed net XIO_RAM_A1: PSRAM.A1@4
- removed net XIO_RAM_A10: PSRAM.A10@25
- removed net XIO_RAM_A11: PSRAM.A11@24
- removed net XIO_RAM_A12: PSRAM.A12@22
- removed net XIO_RAM_A13: PSRAM.A13@21
- removed net XIO_RAM_A14: PSRAM.A14@20
- removed net XIO_RAM_A15: PSRAM.A15@19
- removed net XIO_RAM_A16: PSRAM.A16@18
- removed net XIO_RAM_A17: PSRAM.A17@23
- removed net XIO_RAM_A18: PSRAM.A18@28
- removed net XIO_RAM_A2: PSRAM.A2@3
- removed net XIO_RAM_A3: PSRAM.A3@2
- removed net XIO_RAM_A4: PSRAM.A4@1
- removed net XIO_RAM_A5: PSRAM.A5@44
- removed net XIO_RAM_A6: PSRAM.A6@43
- removed net XIO_RAM_A7: PSRAM.A7@42
- removed net XIO_RAM_A8: PSRAM.A8@27
- removed net XIO_RAM_A9: PSRAM.A9@26
- removed net XIO_RAM_D0: PSRAM.D0@7
- removed net XIO_RAM_D1: PSRAM.D1@8
- removed net XIO_RAM_D10: PSRAM.D10@31
- removed net XIO_RAM_D11: PSRAM.D11@32
- removed net XIO_RAM_D12: PSRAM.D12@35
- removed net XIO_RAM_D13: PSRAM.D13@36
- removed net XIO_RAM_D14: PSRAM.D14@37
- removed net XIO_RAM_D15: PSRAM.D15@38
- removed net XIO_RAM_D2: PSRAM.D2@9
- removed net XIO_RAM_D3: PSRAM.D3@10
- removed net XIO_RAM_D4: PSRAM.D4@13
- removed net XIO_RAM_D5: PSRAM.D5@14
- removed net XIO_RAM_D6: PSRAM.D6@15
- removed net XIO_RAM_D7: PSRAM.D7@16
- removed net XIO_RAM_D8: PSRAM.D8@29
- removed net XIO_RAM_D9: PSRAM.D9@30
- net +3V3: no longer C19.1, C20.1, C52.1, PSRAM.VDD@11, PSRAM.VDD@33
- net GND: no longer C19.2, C20.2, C52.2, PSRAM.GND@12, PSRAM.GND@34
Other:
- note added: "@400"
- note removed: "1 MB PSRAM"
- note removed: "@200"
- note removed: "@216"
- note removed: "PSRAM access time guaranteed at 60ns If we could use SDRAM, could bump the memory to 32MBytes. - does SDRAM refresh impact access time too much ?"
- moved on the sheet: XIO-SDRAM
