File: boards/xio3/xio3.sch (EAGLE design)
At the start: 352 parts, among them J1 12401598E4#2A, Q1 BSS138, Q2 BSS138, Q3 BC817-16LT3G, Q4 BC817-16LT3G, Y2 FA-238 25.0000MB-K3

Commit message: Attempt at 3rd version of board, this time using a COTS FPGA board
Parts:
- removed ADV7125: ADV7125, sjg-analog:ADV7125
- removed A_MUX: TS3A27518EPWR, sjg-logic:TS3A27518E
- removed BOOT_MODE: 209-3MS, special:SW_DIP-3
- removed C1, C34, C43: 10uF, rcl:C-EUC0402K
- removed C10, C100, C106, C113, C114, C115, C116, C117, C118, C119, C120, C121, C122, C123, C124, C125, C126, C127, C128, C129, C13, C130, C131, C132, C133, C134, C137, C138, C16, C167, C168, C169, C170, C171, C172, C19, C2, C20, C21, C22, C23, C24, C25, C26, C27, C28, C29, C3, C31, C32, C33, C35, C38, C39, C4, C40, C45, C5, C57, C6, C60, C61, C62, C63, C64, C65, C66, C67, C68, C69, C7, C70, C71, C72, C8, C80, C87, C88, C9, C96, C98: 0.1uF, rcl:C-EUC0201
- removed C101, C73, C77: 100uF, rcl:C-EUC0805
- removed C102, C108, C59, C74, C75, C76, C78, C79, C82: 4.7uF, rcl:C-EUC0402
- removed C104, C30, C36, C47, C48, C49, C50, C51, C58, C83, C84, C85, C86: 0.47uF, rcl:C-EUC0201
- removed C109, C110, C41: 22uF, rcl:C-EUC0805
- removed C11, C139, C140, C141: 10uF, rcl:C-EUC0805
- removed C111: 0.01uF, rcl:C-EUC0402
- removed C112: 3900pF, rcl:C-EUC0402
- removed C12: 22uF, rcl:C-EUC2012
- removed C135: 120pF, rcl:C-EUC0201
- removed C136, C37, C44, C93: 0.01uF, rcl:C-EUC0201
- removed C14, C15: 16pF, rcl:C-EUC0201
- removed C142: 0.1uF, rcl:C-EUC0402
- removed C143: 1.2nF, rcl:C-EUC0603
- removed C144: 13pF, rcl:C-EUC0805
- removed C145: 560pF, rcl:C-EUC0402
- removed C146: 33uF, rcl:C-EUC0805
- removed C17, C18, C99: 2.2uF, rcl:C-EUC0201
- removed C173, C42, C46, C97: 1uF, rcl:C-EUC0201
- removed C177: 4.7uF, rcl:C-EUC0201
- removed C52: 47uF, rcl:C-EUC0805
- removed D1, D2: BAT54S, diode:BAT54S
- removed DBG0, DBG1, DBG2: YELLOW_LED, microbuilder:LED0603
- removed EXPANSION: (no value), pinhead:PINHD-2X6
- removed EXP_POWER, PEXT_10, PEXT_18: (no value), pinhead:PINHD-1X2
- removed FPGA_1_0: TLV62095, sjg-power:TLV62095
- removed FPGA_CFG: W25Q80DVSNIG, microbuilder:SPIFLASH_SOIC8
- removed FPGA_DONE: LTST-C191KFKT, microbuilder:LED0603
- removed FPGA_PROG: XILINX-JTAG, sjg-con:XILINX-JTAG
- removed H1, H2, H4, H5: MOUNT-HOLE3.2, holes:MOUNT-HOLE3.2
- removed HOST_IO: (no value), pinhead:PINHD-2X20/90
- removed IO_EXP: MCP23S17T-E/SS, sjg-logic:MCP23S17T-E/SS
- removed J1: 12401598E4#2A, usb-c:12401598E4#2A
- removed L1: 1.5uH, rcl:L-EUL5650M
- removed L2: 2.2uH, sjg-inductor:PA4332
- removed L3: 470nH, sjg-power:DFE18SANR47MG0L
- removed LD_0ACT, LD_1ACT, LD_2ACT, LD_3ACT, LD_4ACT: LTST-C191KRKT, led:LEDCHIPLED_0603
- removed LD_7DBG0, LD_7DBG1, LD_7DBG2: IN-S63BTA, led:LEDCHIPLED_0603
- removed LD_AUX, LD_INT, LD_V33: LTST-S270GKT, led:LEDCHIPLED_0603
- removed MUX-HI, MUX-LO: IDTQS3VH257, sjg-logic:IDTQS3VH257
- removed OSC1: 50 MHz oscillator, microbuilder:OSCILLATOR3.2X2.5
- removed PEXT_33: (no value), pinhead:PINHD-2X2
- removed POWER: dc5vin, sjg-power:CONN-POWER-JACK-2.1MM(DC-005)
- removed PSW: NCP380, sjg-power:NCP380
- removed Q1, Q2: BSS138, transistor-small-signal:BSS123
- removed Q3, Q4: BC817-16LT3G, microbuilder:TRANSISTOR_NPN
- removed R1, R24, R5, R53, R72: 0R, rcl:R-EU_R0201
- removed R10: 560R, rcl:R-EU_R0201
- removed R102, R105, R108, R109, R110, R111, R2, R3, R4, R94, R99: 130R, rcl:R-EU_R0402
- removed R112: 59R, rcl:R-EU_R0402
- removed R113, R114, R115, R116, R117, R118: 50R, rcl:R-EU_R0201
- removed R119: 100K, rcl:R-EU_R0201
- removed R120, R121, R59, R81, R82, R83, R84, R85, R88, R89, R90: 10K, rcl:R-EU_R0201
- removed R125, R126, R127: 47K, rcl:R-EU_R0201
- removed R128, R13, R50, R51, R58: 1K, rcl:R-EU_R0201
- removed R129: 499K, rcl:R-EU_R0402
- removed R130: 40.2K, rcl:R-EU_R0402
- removed R131: 160K, rcl:R-EU_R0402
- removed R133: 10.5R, rcl:R-EU_R0402
- removed R134: 48.7K, rcl:R-EU_R0402
- removed R135: 6.04K, rcl:R-EU_R0805
- removed R136: 12K, rcl:R-EU_R0805
- removed R137: 2.67K, rcl:R-EU_R0402
- removed R138: 64.9R, rcl:R-EU_R0402
- removed R139: 105K, rcl:R-EU_R0201
- removed R19, R20, R22: 75R, rcl:R-EU_R0201
- removed R21, R26, R27, R52, R60, R73, R74, R75, R91, R92, R93: 33R, rcl:R-EU_R0201
- removed R23, R69, R70, R71, R78, R79: 4.7K, rcl:R-EU_R0201
- removed R36, R37, R38, R39, R40, R41: 47K, rcl:R-EU_R0402
- removed R54, R55, R57: 2.4K, rcl:R-EU_R0201
- removed R56: 1M, rcl:R-EU_R0402
- removed R66: 200R, rcl:R-EU_R0201
- removed R67, R77: 150R, rcl:R-EU_R0402
- removed R68: 100R, rcl:R-EU_R0402
- removed R76, R80: 330R, rcl:R-EU_R0402
- removed RESET_S7: Tac-switch, SparkFun:TAC_SWITCHPTH
- removed RESET_XIO: TAC_SWITCH, SparkFun:TAC_SWITCHPTH
- removed SDRAM: IS42S32160F-7TLI, sjg-sdram:IS42S32160F-7TLI
- removed SD_SLOT: 5025700893, j_microsd_molex_5025700893:MICROSD_MOLEX_5025700893
- removed SPI_DBG: (no value), pinhead:PINHD-1X5
- removed U$6, U$7, U$8: 74LVC1T45GWSOT866, sjg-logic:74LVC1T45GWSOT866
- removed USB: MINI-USB-UX60-MB-5ST, con-hirose:MINI-USB-UX60-MB-5ST
- removed USB_ESD: PUSB2X4YH, sjg-isolation:PUSB2X4YH
- removed VGA: 15-way D, SparkFun-Connectors:DB15
- removed VREG_18: TPS62087RLTR, sjg-ti:TPS62087RLTR
- removed VREG_33: LM21212, sjg-power:LM21212
- removed VREG_MON: TPS3808G33DBVR, sjg-power:TPS3808DBVR
- removed VREG_VGA: AD1580ARTZ, sjg-analog:AD1580ARTZ
- removed XC7S25: XC7S25, sjg-xilinx:XC7S25
- removed XIO: STM32H743-XIO, sjg-stm32:STM32H743-XIO
- removed XIO-SWD: XIO_JTAG, sjg-stm32:STM_DEBUG
- removed XSPI5_DBG, XSPI6_DBG: (no value), pinhead:PINHD-1X3
- removed Y2: FA-238 25.0000MB-K3, microbuilder:CRYSTALTHIN
- added H3, H6, H7, H8: MOUNT-HOLE4.1, holes:MOUNT-HOLE4.1
- added U$1: QM_A35T, sjg-fpga:QM_A35T
- added U$2: DB15, SparkFun-Connectors:DB15
Connections:
- removed net !ADDR_VALID_READ!: XC7S25-BANK34.IO_L11P_T1_SRCC_34@D1, XIO-HOST.PC1@M2
- removed net !ADDR_VALID_WRITE!: XC7S25-BANK34.IO_L11N_T1_SRCC_34@C1, XIO-HOST.PC2@M3
- removed net !GEN_CCTL!: LVL_AHI.A6@8, XC7S25-BANK34.IO_L12N_T1_MRCC_34@F4
- removed net !GEN_S4!: LVL_AHI.A7@9, XC7S25-BANK34.IO_L13N_T2_MRCC_34@H3
- removed net !GEN_S5!: LVL_AHI.A8@10, XC7S25-BANK34.IO_L14P_T2_SRCC_34@H2
- removed net !IO_EXP_IRQ!: IO_EXP.INTA@20, IO_EXP.INTB@19, XIO-SPI.PE3@D3
- removed net !IO_EXP_SEL!: IO_EXP.!CS!@11, XIO-SPI.PH2@N2
- removed net !MR!: C136.1, RESET_XIO.1, RESET_XIO.2, VREG_MON.!MR!@3
- removed net !RESET!: C98.1, IO_EXP.!RESET!@18, R89.2, VREG_MON.!RESET!@1, XIO-POWER.!RST!@K1, XIO-SWD.RESET@10
- removed net !SDRAM_CAS!: SDRAM.!CAS!@18, XIO-SDRAM.PG15@D6
- removed net !SDRAM_RAS!: SDRAM.!RAS!@19, XIO-SDRAM.PF11@T7
- removed net !SDRAM_WE!: SDRAM.!WE!@17, XIO-SDRAM.PH5@P4
- removed net !SPI_IRQ!: XC7S25-BANK34.IO_L22N_T3_34@L2, XIO-SPI.PE4@D2
- removed net AGND: C1.2, C13.2, R72.2, XIO-POWER.VREF-@N1, XIO-POWER.VSSA@P1
- removed net BOOT0: R1.1, R5.2, XIO-POWER.BOOT0@E8
- removed net BOOT_M0: BOOT_MODE.1, R127.1, XC7S25-CFG.M0_0@M7
- removed net BOOT_M1: BOOT_MODE.2, R126.1, XC7S25-CFG.M1_0@M8
- removed net BOOT_M2: BOOT_MODE.3, R125.1, XC7S25-CFG.M2_0@M9
- removed net CART_!CCTL!: CARTRIDGE.!CCTL!@15, LVL_AHI.B6@16
- removed net CART_!S4!: CARTRIDGE.!S4!@1, LVL_AHI.B7@15
- removed net CART_!S5!: CARTRIDGE.!S5!@12, LVL_AHI.B8@14
- removed net CART_A0: CARTRIDGE.A0@5, LVL_ALO.B1@21
- removed net CART_A1: CARTRIDGE.A1@4, LVL_ALO.B2@20
- removed net CART_A10: CARTRIDGE.A10@P, LVL_AHI.B3@19
- removed net CART_A11: CARTRIDGE.A11@N, LVL_AHI.B4@18
- removed net CART_A12: CARTRIDGE.A12@K, LVL_AHI.B5@17
- removed net CART_A2: CARTRIDGE.A2@3, LVL_ALO.B3@19
- removed net CART_A3: CARTRIDGE.A3@2, LVL_ALO.B4@18
- removed net CART_A4: CARTRIDGE.A4@C, LVL_ALO.B5@17
- removed net CART_A5: CARTRIDGE.A5@D, LVL_ALO.B6@16
- removed net CART_A6: CARTRIDGE.A6@E, LVL_ALO.B7@15
- removed net CART_A7: CARTRIDGE.A7@F, LVL_ALO.B8@14
- removed net CART_A8: CARTRIDGE.A8@H, LVL_AHI.B1@21
- removed net CART_A9: CARTRIDGE.A9@J, LVL_AHI.B2@20
- removed net CART_CLK: CARTRIDGE.B02@S, U$5.B@4
- removed net CART_D0: CARTRIDGE.D0@10, LVL_D.B1@21
- removed net CART_D1: CARTRIDGE.D1@9, LVL_D.B2@20
- removed net CART_D2: CARTRIDGE.D2@8, LVL_D.B3@19
- removed net CART_D3: CARTRIDGE.D3@L, LVL_D.B4@18
- removed net CART_D4: CARTRIDGE.D4@6, LVL_D.B5@17
- removed net CART_D5: CARTRIDGE.D5@7, LVL_D.B6@16
- removed net CART_D6: CARTRIDGE.D6@11, LVL_D.B7@15
- removed net CART_D7: CARTRIDGE.D7@M, LVL_D.B8@14
- removed net CART_R/!W!: CARTRIDGE.R/!W!@R, U$6.B@4
- removed net CART_RD4: U$7.B@4, XC7S25-BANK34.IO_L14N_T2_SRCC_34@H1
- removed net CART_RD5: U$8.B@4, XC7S25-BANK34.IO_L15P_T2_DQS_34@J2
- removed net EXT_IO0: EXPANSION.8, IO_EXP.GPB6@7
- removed net EXT_IO1: EXPANSION.10, IO_EXP.GPB7@8
- removed net FLASH_CLK: A_MUX.NC1@2, R52.2
- removed net FLASH_CS: A_MUX.NC4@21, R57.1, XC7S25-CFG.IO_L6P_T0_FCS_B_14@C11
- removed net FLASH_D0: A_MUX.NC2@1, R60.2
- removed net FLASH_D1: A_MUX.NC3@23, XC7S25-CFG.IO_L1N_T0_D01_DIN_14@B12
- removed net FLASH_D2: A_MUX.NC5@19, R55.1, XC7S25-CFG.IO_L2P_T0_D02_14@D10
- removed net FLASH_D3: A_MUX.NC6@22, R54.1, XC7S25-CFG.IO_L2N_T0_D03_14@C10
- removed net FPGA_EXT0: EXPANSION.2, XC7S25-BANK34.IO_L16N_T2_34@K3
- removed net FPGA_EXT1: EXPANSION.3, XC7S25-BANK34.IO_L17P_T2_34@J4
- removed net FPGA_EXT2: EXPANSION.4, XC7S25-BANK34.IO_L17N_T2_34@J3
- removed net FPGA_EXT3: EXPANSION.5, XC7S25-BANK34.IO_L18P_T2_34@M1
- removed net FPGA_EXT4: EXPANSION.6, XC7S25-BANK34.IO_L18N_T2_34@L1
- removed net FPGA_EXT5: EXPANSION.7, XC7S25-BANK34.IO_L19P_T3_34@M3
- removed net HOST_CTL0: HOST_IO.2, XC7S25-BANK14.IO_L23P_T3_D19_14@N10
- removed net HOST_CTL1: HOST_IO.4, XC7S25-BANK14.IO_L23N_T3_D18_14@N11
- removed net HOST_DIR0: HOST_IO.22, LVL_D.DIR@2, XC7S25-BANK34.IO_0_34@B6
- removed net HOST_DIR1: HOST_IO.24, XC7S25-BANK34.IO_L1P_T0_34@D3
- removed net HOST_DIR2: HOST_IO.26, XC7S25-BANK34.IO_L1N_T0_34@C3
- removed net HOST_DIR3: HOST_IO.28, XC7S25-BANK34.IO_L2P_T0_34@A4
- removed net HOST_DIR4: HOST_IO.30, XC7S25-BANK34.IO_L2N_T0_34@A3
- removed net LCD_B0: ADV7125.B0@16, XIO-LCD.PJ12@D11
- removed net LCD_B1: ADV7125.B1@17, XIO-LCD.PJ13@E10
- removed net LCD_B2: ADV7125.B2@18, XIO-LCD.PJ14@D10
- removed net LCD_B3: ADV7125.B3@19, XIO-LCD.PJ15@B10
- removed net LCD_B4: ADV7125.B4@20, XIO-LCD.PK3@C8
- removed net LCD_B5: ADV7125.B5@21, XIO-LCD.PK4@B8
- removed net LCD_B6: ADV7125.B6@22, XIO-LCD.PK5@A8
- removed net LCD_B7: ADV7125.B7@23, XIO-LCD.PK6@C7
- removed net LCD_BLANK: ADV7125.!BLANK!@11, XIO-LCD.PK7@D7
- removed net LCD_CLK: ADV7125.CLOCK@24, XIO-LCD.PG7@F16
- removed net LCD_G0: ADV7125.G0@3, XIO-LCD.PJ7@N14
- removed net LCD_G1: ADV7125.G1@4, XIO-LCD.PJ8@N13
- removed net LCD_G2: ADV7125.G2@5, XIO-LCD.PJ9@M14
- removed net LCD_G3: ADV7125.G3@6, XIO-LCD.PJ10@L14
- removed net LCD_G4: ADV7125.G4@7, XIO-LCD.PJ11@K14
- removed net LCD_G5: ADV7125.G5@8, XIO-LCD.PK0@J14
- removed net LCD_G6: ADV7125.G6@9, XIO-LCD.PK1@J15
- removed net LCD_G7: ADV7125.G7@10, XIO-LCD.PK2@H17
- removed net LCD_HS: Q2.S, XIO-LCD.PI12@H1
- removed net LCD_R0: ADV7125.R0@41, XIO-LCD.PI15@P5
- removed net LCD_R1: ADV7125.R1@42, XIO-LCD.PJ0@N6
- removed net LCD_R2: ADV7125.R2@43, XIO-LCD.PJ1@P6
- removed net LCD_R3: ADV7125.R3@44, XIO-LCD.PJ2@T6
- removed net LCD_R4: ADV7125.R4@45, XIO-LCD.PJ3@U6
- removed net LCD_R5: ADV7125.R5@46, XIO-LCD.PJ4@U7
- removed net LCD_R6: ADV7125.R6@47, XIO-LCD.PJ5@R12
- removed net LCD_R7: ADV7125.R7@48, XIO-LCD.PJ6@N15
- removed net LCD_VS: Q1.S, XIO-LCD.PI13@H2
- removed net LX_CLK: OSC1.OUT, XC7S25-BANK34.IO_L12P_T1_MRCC_34@G4
- removed net LX_MISC: J1.CC1, XC7S25-BANK14.IO_25_14@M10
- removed net LX_RC_N: J1.SSRXP1, XC7S25-BANK14.IO_L24N_T3_D16_14@P11
- removed net LX_RC_P: J1.SSRXN1, XC7S25-BANK14.IO_L24P_T3_D17_14@P10
- removed net LX_RD_N: J1.SSTXP2, XC7S25-BANK14.IO_L14N_T2_SRCC_14@H14
- removed net LX_RD_P: J1.SSTXN2, XC7S25-BANK14.IO_L14P_T2_SRCC_14@H13
- removed net LX_TC_N: J1.DN1, R113.1, XC7S25-BANK14.IO_L21N_T3_DQS_D22_14@M14
- removed net LX_TC_P: J1.DP1, R114.1, XC7S25-BANK14.IO_L21P_T3_DQS_14@N14
- removed net LX_TD0_N: J1.SSTXN1, R115.1, XC7S25-BANK14.IO_L22N_T3_D20_14@P13
- removed net LX_TD0_P: J1.SSTXP1, R116.1, XC7S25-BANK14.IO_L22P_T3_D21_14@P12
- removed net LX_TD1_N: J1.SSRXN2, R117.1, XC7S25-BANK14.IO_L18N_T2_D27_14@J14
- removed net LX_TD1_P: J1.SSRXP2, R118.1, XC7S25-BANK14.IO_L18P_T2_D28_14@J13
- removed net N$1: PSW.EN@3, XIO-USB.PA15@A14
- removed net N$10: ADV7125.!PSAVE!@38, R23.1
- removed net N$102: LD_4ACT.A, R108.2
- removed net N$103: LD_7DBG0.A, R109.2
- removed net N$104: LD_7DBG1.A, R110.2
- removed net N$105: LD_7DBG2.A, R111.2
- removed net N$106: LD_V33.A, R112.2
- removed net N$108: C143.1, C144.1, VREG_33.COMP@18
- removed net N$109: C143.2, R135.2
- removed net N$110: C144.2, R135.1, R136.2, R137.1, R138.2, VREG_33.FB@19
- removed net N$113: C145.2, R138.1
- removed net N$12: DBG0.A, R2.2
- removed net N$13: DBG0.C, XIO-LED.PD11@R15
- removed net N$14: DBG1.C, XIO-LED.PD12@R16
- removed net N$15: DBG2.C, XIO-LED.PD13@R17
- removed net N$16: DBG1.A, R3.2
- removed net N$17: ADV7125.RSET@37, R10.2
- removed net N$18: ADV7125.!SYNC!@12, R24.2
- removed net N$19: DBG2.A, R4.2
- removed net N$2: R121.2, SDRAM.CKE@67
- removed net N$3: R60.1, XC7S25-CFG.IO_L1P_T0_D00_MOSI_14@B11
- removed net N$4: A_MUX.COM1@4, FPGA_CFG.SCK
- removed net N$5: OSC1.INH, R58.2
- removed net N$50: BOOT_MODE.4, BOOT_MODE.5, BOOT_MODE.6, R128.2
- removed net N$51: R52.1, XC7S25-CFG.CCLK_0@A8
- removed net N$55: R66.1, R68.2, XC7S25-CFG.DONE_0@P9
- removed net N$56: FPGA_DONE.A, R68.1
- removed net N$57: R26.2, XIO-SPI.PE2@C3
- removed net N$58: CARTRIDGE.RD4@A, U$7.A@3
- removed net N$59: CARTRIDGE.RD5@14, U$8.A@3
- removed net N$6: ADV7125.VREF@36, C46.1, R13.1, VREG_VGA.V+@1
- removed net N$60: C135.1, VREG_MON.CT@4
- removed net N$61: R27.2, XIO-SPI.PE6@E5
- removed net N$62: A_MUX.COM2@6, FPGA_CFG.MOSI
- removed net N$63: A_MUX.COM3@7, FPGA_CFG.MISO
- removed net N$64: C111.1, FPGA_1_0.CP@7
- removed net N$65: PSW.!FLAG!@4, R119.2, XIO-USB.PD7@C11
- removed net N$66: A_MUX.COM4@9, FPGA_CFG.SSEL
- removed net N$67: A_MUX.COM5@10, FPGA_CFG.#WP/IO2
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Other:
- note removed: "!MR! has internal pull-up to VDD"
- note removed: "(Load Cap 10pF, stray Cap 2pF)"
- note removed: "0.035 mm 0.12 mm 10 mil 7 mil 4.4 90.5 ohms"
- note removed: "0.035 mm 0.12 mm 8 mil 4.4 50.2 ohms"
- note removed: "100uF 47uF 4.7uF 0.47uF"
- note removed: "100uF caps can be placed anywhere others within 2 electrical inches of part"
- note removed: "5v-in is ok to NC"
- note removed: ": GRM21BR60J107ME15L (0805) : GRM21BR60J476ME15L (0805) : GRM155R60J475ME87D (0402) : GRM033R60J474KE90D (0201)"
- note removed: "Add termination resistors close to source"
- note removed: "Amber LED"
- note removed: "Bank 0 / Flash Config"
- note removed: "Boot mode"
- note removed: "Bypass cap number and capacitance taken from UG483"
- note removed: "Bypass caps for muxes"
- note removed: "C.res1 = C.res2 = 2(C.load - C.stray)"
- note removed: "C108 will fail the BOM processing as being of different type than all the other 4.7uF caps. This is expected, since C108 is higher voltage-rated"
- note removed: "C11 C12 L3 R56"
- note removed: "C139 C140 C141 C142 C143 C144 C145 C146 R133 R134 R135 R136 R137 R138 R139 L2"
- note removed: "Caps placed close to VCAP pins"
- note removed: "Caps placed close to VDDA pin"
- note removed: "Debug LEDs"
- note removed: "Default (NC) is that the FPGA has control over the SPI flash. If the STM pulls SPI_MUX_IN high, it gains control"
- note removed: "Direction control"
- note removed: "Done goes high once configuration completes"
- note removed: "FLASH_CLK impedance matching"
- note removed: "FPGA Bank 14"
- note removed: "FPGA Bank 34"
- note removed: "FPGA SPI, @ 100MHz"
- note removed: "FPGA decodes bus and handles timings. Sends IRQ when bus is valid to read/write"
- note removed: "FPGA power"
- note removed: "FPGA power supplies"
- note removed: "FPGA to STM32 Host interface"
- note removed: "Filter on VDDA"
- note removed: "Green LED"
- note removed: "Ground-loop caps"
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
Commit message: Start to connect up the cartridge port
Parts:
- added J1: POWER_JACKPTH, SparkFun:POWER_JACKPTH
- added U$3: MINI-SAS, sjg-con:MINI-SAS
- added U$4, U$6, U$7, U$8, U$9: 74LVC1T45GWSOT866, sjg-logic:74LVC1T45GWSOT866
Connections:
- new net !H_CCTL!: CARTRIDGE.!CCTL!@15
- new net !H_EXTSEL!: U$3.B13
- new net !H_HALT!: U$3.A14
- new net !H_IRQ!: U$3.B14
- new net !H_MPD!: U$3.A15
- new net !H_RST!: U$3.A17
- new net !H_S4!: CARTRIDGE.!S4!@1
- new net !H_S5!: CARTRIDGE.!S5!@12
- new net H_A0: CARTRIDGE.A0@5, LVL_ALO.B1@21, U$3.A1
- new net H_A1: CARTRIDGE.A1@4, LVL_ALO.B2@20, U$3.B1
- new net H_A10: CARTRIDGE.A10@P, LVL_AHI.B3@19, U$3.A6
- new net H_A11: CARTRIDGE.A11@N, LVL_AHI.B4@18, U$3.B6
- new net H_A12: CARTRIDGE.A12@K, LVL_AHI.B5@17, U$3.A7
- new net H_A13: LVL_AHI.B6@16, U$3.B7
- new net H_A14: LVL_AHI.B7@15, U$3.A8
- new net H_A15: LVL_AHI.B8@14, U$3.B8
- new net H_A2: CARTRIDGE.A2@3, LVL_ALO.B3@19, U$3.A2
- new net H_A3: CARTRIDGE.A3@2, LVL_ALO.B4@18, U$3.B2
- new net H_A4: CARTRIDGE.A4@C, LVL_ALO.B5@17, U$3.A3
- new net H_A5: CARTRIDGE.A5@D, LVL_ALO.B6@16, U$3.B3
- new net H_A6: CARTRIDGE.A6@E, LVL_ALO.B7@15, U$3.A4
- new net H_A7: CARTRIDGE.A7@F, LVL_ALO.B8@14, U$3.B4
- new net H_A8: CARTRIDGE.A8@H, LVL_AHI.B1@21, U$3.A5
- new net H_A9: CARTRIDGE.A9@J, LVL_AHI.B2@20, U$3.B5
- new net H_CLK: CARTRIDGE.B02@S, U$3.A9
- new net H_D0: CARTRIDGE.D0@10, LVL_D.B1@21, U$3.B9
- new net H_D1: CARTRIDGE.D1@9, LVL_D.B2@20, U$3.A10
- new net H_D2: CARTRIDGE.D2@8, LVL_D.B3@19, U$3.B10
- new net H_D3: CARTRIDGE.D3@L, LVL_D.B4@18, U$3.A11
- new net H_D4: CARTRIDGE.D4@6, LVL_D.B5@17, U$3.B11
- new net H_D5: CARTRIDGE.D5@7, LVL_D.B6@16, U$3.A12
- new net H_D6: CARTRIDGE.D6@11, LVL_D.B7@15, U$3.B12
- new net H_D7: CARTRIDGE.D7@M, LVL_D.B8@14, U$3.A13
- new net H_R/!W!: CARTRIDGE.R/!W!@R, U$3.B17
- new net H_RD4: CARTRIDGE.RD4@A, U$3.B15
- new net H_RD5: CARTRIDGE.RD5@14, U$3.A16
- new net H_REF: U$3.B16
- net +3V3: now also U$4.DIR@5, U$4.VCCA@1, U$6.DIR@5, U$6.VCCA@1, U$7.DIR@5, U$7.VCCA@1, U$8.DIR@5, U$8.VCCA@1, U$9.DIR@5, U$9.VCCA@1
- net +5V: now also U$4.VCCB@6, U$6.VCCB@6, U$7.VCCB@6, U$8.VCCB@6, U$9.VCCB@6
- net GND: now also U$3.SHIELD, U$4.GND@2, U$6.GND@2, U$7.GND@2, U$8.GND@2, U$9.GND@2
Other:
- note added: "Artix 7 XC7A35T-1 BGA256"
- note removed: "Artix 7 XC735T-1 BGA256"

Commit message: Before deciding which signals to drop for S4,S5
Parts:
- removed J1: POWER_JACKPTH, SparkFun:POWER_JACKPTH
- removed LD_0P: SML-D12D1WT86, led:LEDCHIPLED_0603
- removed R87: 59R, rcl:R-EU_R0402
- added C1, C10, C11, C12, C13, C134, C14, C15, C16, C17, C18, C2, C3, C4, C5, C57, C6, C60, C61, C62, C63, C64, C65, C66, C67, C68, C69, C7, C70, C71, C72, C8, C9: 0.1uF, rcl:C-EUC0201
- added C41: 22uF, rcl:C-EUC0805
- added C42: 1uF, rcl:C-EUC0201
- added C43: 10uF, rcl:C-EUC0402K
- added JP1: (no value), pinhead:PINHD-2X25
- added JP2: (no value), pinhead:PINHD-2X10
- added JP3: (no value), pinhead:PINHD-2X8
- added LD_0P1: SML-D12D1WT86, led:LEDCHIPLED_0603
- added POWER: dc5vin, sjg-power:CONN-POWER-JACK-2.1MM(DC-005)
- added R1, R10, R13, R19, R2, R20, R21, R22, R23, R24, R25, R26, R3, R4, R5: 10K, rcl:R-EU_R0201
- added R27: 59R, rcl:R-EU_R0402
- added R28, R29: 100R, rcl:R-EU_R0201
- added R36, R37, R38, R39, R40, R41: 4K7, rcl:R-EU_R0402
- added RN1, RN5, RN8: 1K, sjg-resistor:ACAS0612
- added RN10, RN11, RN2, RN3, RN4, RN6, RN7, RN9: 2K, sjg-resistor:ACAS0612
- added SD_SLOT: 5025700893, j_microsd_molex_5025700893:MICROSD_MOLEX_5025700893
- added U$11, U$12, U$13, U$14, U$15, U$16, U$17: 74LVC1T45GWSOT866, sjg-logic:74LVC1T45GWSOT866
Connections:
- removed net !H_CCTL!: CARTRIDGE.!CCTL!@15
- removed net !H_EXTSEL!: U$3.B13
- removed net !H_HALT!: U$3.A14
- removed net !H_IRQ!: U$3.B14
- removed net !H_MPD!: U$3.A15
- removed net !H_RST!: U$3.A17
- removed net !H_S4!: CARTRIDGE.!S4!@1
- removed net !H_S5!: CARTRIDGE.!S5!@12
- removed net HOST_!EXTSEL!: SLOT0.B26, SLOT1.B26, SLOT2.B26, SLOT3.B26, SLOT4.B26
- removed net HOST_!HALT!: SLOT0.B27, SLOT1.B27, SLOT2.B27, SLOT3.B27, SLOT4.B27
- removed net HOST_!IRQ!: SLOT0.B28, SLOT1.B28, SLOT2.B28, SLOT3.B28, SLOT4.B28
- removed net HOST_!MPD!: SLOT0.B29, SLOT1.B29, SLOT2.B29, SLOT3.B29, SLOT4.B29
- removed net HOST_!REF!: SLOT0.B30, SLOT1.B30, SLOT2.B30, SLOT3.B30, SLOT4.B30
- removed net HOST_!RST!: SLOT0.B31, SLOT1.B31, SLOT2.B31, SLOT3.B31, SLOT4.B31
- removed net HOST_A0: SLOT0.A8, SLOT1.A8, SLOT2.A8, SLOT3.A8, SLOT4.A7
- removed net HOST_A1: SLOT0.A9, SLOT1.A9, SLOT2.A9, SLOT3.A9, SLOT4.A8
- removed net HOST_A10: SLOT0.A18, SLOT1.A18, SLOT2.A18, SLOT3.A18, SLOT4.A17
- removed net HOST_A11: SLOT0.A19, SLOT1.A19, SLOT2.A19, SLOT3.A19, SLOT4.A18
- removed net HOST_A12: SLOT0.A20, SLOT1.A20, SLOT2.A20, SLOT3.A20, SLOT4.A19
- removed net HOST_A13: SLOT0.A21, SLOT1.A21, SLOT2.A21, SLOT3.A21, SLOT4.A20
- removed net HOST_A14: SLOT0.A22, SLOT1.A22, SLOT2.A22, SLOT3.A22, SLOT4.A21
- removed net HOST_A15: SLOT0.A23, SLOT1.A23, SLOT2.A23, SLOT3.A23, SLOT4.A22
- removed net HOST_A2: SLOT0.A10, SLOT1.A10, SLOT2.A10, SLOT3.A10, SLOT4.A9
- removed net HOST_A3: SLOT0.A11, SLOT1.A11, SLOT2.A11, SLOT3.A11, SLOT4.A10
- removed net HOST_A4: SLOT0.A12, SLOT1.A12, SLOT2.A12, SLOT3.A12, SLOT4.A11
- removed net HOST_A5: SLOT0.A13, SLOT1.A13, SLOT2.A13, SLOT3.A13, SLOT4.A12
- removed net HOST_A6: SLOT0.A14, SLOT1.A14, SLOT2.A14, SLOT3.A14, SLOT4.A13
- removed net HOST_A7: SLOT0.A15, SLOT1.A15, SLOT2.A15, SLOT3.A15, SLOT4.A14
- removed net HOST_A8: SLOT0.A16, SLOT1.A16, SLOT2.A16, SLOT3.A16, SLOT4.A15
- removed net HOST_A9: SLOT0.A17, SLOT1.A17, SLOT2.A17, SLOT3.A17, SLOT4.A16
- removed net HOST_CLK: SLOT0.A24, SLOT1.A24, SLOT2.A24, SLOT3.A24, SLOT4.A23
- removed net HOST_D0: SLOT0.A25, SLOT1.A25, SLOT2.A25, SLOT3.A25, SLOT4.A24
- removed net HOST_D1: SLOT0.A26, SLOT1.A26, SLOT2.A26, SLOT3.A26, SLOT4.A25
- removed net HOST_D2: SLOT0.A27, SLOT1.A27, SLOT2.A27, SLOT3.A27, SLOT4.A26
- removed net HOST_D3: SLOT0.A28, SLOT1.A28, SLOT2.A28, SLOT3.A28, SLOT4.A27
- removed net HOST_D4: SLOT0.A29, SLOT1.A29, SLOT2.A29, SLOT3.A29, SLOT4.A28
- removed net HOST_D5: SLOT0.A30, SLOT1.A30, SLOT2.A30, SLOT3.A30, SLOT4.A29
- removed net HOST_D6: SLOT0.A31, SLOT1.A31, SLOT2.A31, SLOT3.A31, SLOT4.A30
- removed net HOST_D7: SLOT0.A32, SLOT1.A32, SLOT2.A32, SLOT3.A32, SLOT4.A31
- removed net HOST_R/!W!: SLOT0.B32, SLOT1.B32, SLOT2.B32, SLOT3.B32, SLOT4.B32
- removed net H_A0: CARTRIDGE.A0@5, LVL_ALO.B1@21, U$3.A1
- removed net H_A1: CARTRIDGE.A1@4, LVL_ALO.B2@20, U$3.B1
- removed net H_A10: CARTRIDGE.A10@P, LVL_AHI.B3@19, U$3.A6
- removed net H_A11: CARTRIDGE.A11@N, LVL_AHI.B4@18, U$3.B6
- removed net H_A12: CARTRIDGE.A12@K, LVL_AHI.B5@17, U$3.A7
- removed net H_A13: LVL_AHI.B6@16, U$3.B7
- removed net H_A14: LVL_AHI.B7@15, U$3.A8
- removed net H_A15: LVL_AHI.B8@14, U$3.B8
- removed net H_A2: CARTRIDGE.A2@3, LVL_ALO.B3@19, U$3.A2
- removed net H_A3: CARTRIDGE.A3@2, LVL_ALO.B4@18, U$3.B2
- removed net H_A4: CARTRIDGE.A4@C, LVL_ALO.B5@17, U$3.A3
- removed net H_A5: CARTRIDGE.A5@D, LVL_ALO.B6@16, U$3.B3
- removed net H_A6: CARTRIDGE.A6@E, LVL_ALO.B7@15, U$3.A4
- removed net H_A7: CARTRIDGE.A7@F, LVL_ALO.B8@14, U$3.B4
- removed net H_A8: CARTRIDGE.A8@H, LVL_AHI.B1@21, U$3.A5
- removed net H_A9: CARTRIDGE.A9@J, LVL_AHI.B2@20, U$3.B5
- removed net H_CLK: CARTRIDGE.B02@S, U$3.A9
- removed net H_D0: CARTRIDGE.D0@10, LVL_D.B1@21, U$3.B9
- removed net H_D1: CARTRIDGE.D1@9, LVL_D.B2@20, U$3.A10
- removed net H_D2: CARTRIDGE.D2@8, LVL_D.B3@19, U$3.B10
- removed net H_D3: CARTRIDGE.D3@L, LVL_D.B4@18, U$3.A11
- removed net H_D4: CARTRIDGE.D4@6, LVL_D.B5@17, U$3.B11
- removed net H_D5: CARTRIDGE.D5@7, LVL_D.B6@16, U$3.A12
- removed net H_D6: CARTRIDGE.D6@11, LVL_D.B7@15, U$3.B12
- removed net H_D7: CARTRIDGE.D7@M, LVL_D.B8@14, U$3.A13
- removed net H_R/!W!: CARTRIDGE.R/!W!@R, U$3.B17
- removed net H_RD4: CARTRIDGE.RD4@A, U$3.B15
- removed net H_RD5: CARTRIDGE.RD5@14, U$3.A16
- removed net H_REF: U$3.B16
- removed net N$82: LD_0P.A, R87.2
- removed net SBUS12_CTL0: SLOT0.B8, SLOT1.B8
- removed net SBUS12_CTL1: SLOT0.B9, SLOT1.B9
- removed net SBUS12_CTL2: SLOT0.B10, SLOT1.B10
- removed net SBUS12_CTL3: SLOT0.B11, SLOT1.B11
- removed net SBUS12_CTL4: SLOT0.B12, SLOT1.B12
- removed net SBUS12_D0: SLOT0.B18, SLOT1.B18
- removed net SBUS12_D1: SLOT0.B19, SLOT1.B19
- removed net SBUS12_D2: SLOT0.B20, SLOT1.B20
- removed net SBUS12_D3: SLOT0.B21, SLOT1.B21
- removed net SBUS12_D4: SLOT0.B22, SLOT1.B22
- removed net SBUS12_D5: SLOT0.B23, SLOT1.B23
- removed net SBUS12_D6: SLOT0.B24, SLOT1.B24
- removed net SBUS12_D7: SLOT0.B25, SLOT1.B25
- removed net SBUS34_CTL0: SLOT2.B8, SLOT3.B8
- removed net SBUS34_CTL1: SLOT2.B9, SLOT3.B9
- removed net SBUS34_CTL2: SLOT2.B10, SLOT3.B10
- removed net SBUS34_CTL3: SLOT2.B11, SLOT3.B11
- removed net SBUS34_CTL4: SLOT2.B12, SLOT3.B12
- removed net SBUS34_D0: SLOT2.B18, SLOT3.B18
- removed net SBUS34_D1: SLOT2.B19, SLOT3.B19
- removed net SBUS34_D2: SLOT2.B20, SLOT3.B20
- removed net SBUS34_D3: SLOT2.B21, SLOT3.B21
- removed net SBUS34_D4: SLOT2.B22, SLOT3.B22
- removed net SBUS34_D5: SLOT2.B23, SLOT3.B23
- removed net SBUS34_D6: SLOT2.B24, SLOT3.B24
- removed net SBUS34_D7: SLOT2.B25, SLOT3.B25
- removed net SPI_CLK: SLOT0.B17, SLOT1.B17, SLOT2.B17, SLOT3.B17, SLOT4.B17
- removed net SPI_IRQ0: SLOT0.B14
- removed net SPI_IRQ1: SLOT1.B14
- removed net SPI_IRQ2: SLOT2.B14
- removed net SPI_IRQ3: SLOT3.B14
- removed net SPI_IRQ4: SLOT4.B14
- removed net SPI_MISO: SLOT0.B16, SLOT1.B16, SLOT2.B16, SLOT3.B16, SLOT4.B16
- removed net SPI_MOSI: SLOT0.B15, SLOT1.B15, SLOT2.B15, SLOT3.B15, SLOT4.B15
- removed net SPI_SS0: SLOT0.B13
- removed net SPI_SS1: SLOT1.B13
- removed net SPI_SS2: SLOT2.B13
- removed net SPI_SS3: SLOT3.B13
- removed net SPI_SS4: SLOT4.B13
- new net !HI_CCTL!: CARTRIDGE.!CCTL!@15, JP1.34, U$13.B@4, U$3.A18
- new net !HI_EXTSEL!: JP1.36, U$3.B13, U$5.B@4
- new net !HI_HALT!: JP1.39, U$3.A14, U$8.B@4
- new net !HI_IRQ!: JP1.37, U$3.B14, U$6.B@4
- new net !HI_MPD!: JP1.38, U$3.A15, U$4.B@4
- new net !HI_REF!: JP1.40, U$3.B16, U$7.B@4
- new net !HI_RST!: JP1.32, U$17.B@4, U$3.A17
- new net !HI_S4!: CARTRIDGE.!S4!@1, JP1.8, U$12.B@4
- new net !HI_S5!: CARTRIDGE.!S5!@12, JP1.30, U$11.B@4
- new net !LO_CCTL!: SLOT0.A27, SLOT1.A27, SLOT2.A27, SLOT3.A27, SLOT4.A27, U$13.A@3, U$1G$1.BANK14_R10@34
- new net !LO_EXTSEL!: SLOT0.A29, SLOT1.A29, SLOT2.A29, SLOT3.A29, SLOT4.A29, U$1G$1.BANK14_M6@44, U$5.A@3
- new net !LO_HALT!: SLOT0.A30, SLOT1.A30, SLOT2.A30, SLOT3.A30, SLOT4.A30, U$1G$1.BANK34_L5@45, U$8.A@3
- new net !LO_IRQ!: SLOT0.A31, SLOT1.A31, SLOT2.A31, SLOT3.A31, SLOT4.A31, U$1G$1.BANK34_P5@46, U$6.A@3
- new net !LO_MPD!: SLOT0.A32, SLOT1.A32, SLOT2.A32, SLOT3.A32, SLOT4.A32, U$1G$1.BANK34_T4@47, U$4.A@3
- new net !LO_REF!: SLOT0.B17, SLOT1.B17, SLOT2.B17, SLOT3.B17, SLOT4.B17, U$1G$1.BANK34_T2@50, U$7.A@3
- new net !LO_RST!: SLOT0.B18, SLOT1.B18, SLOT2.B18, SLOT3.B18, SLOT4.B18, U$17.A@3, U$1G$1.BANK34_R2@51
- new net !LO_S4!: SLOT0.B20, SLOT1.B20, SLOT2.B20, SLOT3.B20, SLOT4.B20, U$12.A@3, U$1G$1.BANK34_M5@53
- new net !LO_S5!: SLOT0.B21, SLOT1.B21, SLOT2.B21, SLOT3.B21, SLOT4.B21, U$11.A@3, U$1G$1.BANK34_N4@54
- new net DIR_A: LVL_AHI.DIR@2, LVL_ALO.DIR@2, R26.1, U$1G$1.BANK34_P4@55
- new net DIR_CCTL: R1.1, U$13.DIR@5, U$1G$1.BANK34_P3@56
- new net DIR_CLK: R2.1, U$15.DIR@5, U$1G$1.BANK34_N1@57
- new net DIR_D: LVL_D.DIR@2, R25.1, U$1G$1.BANK34_P1@58
- new net DIR_EXTSEL: R3.1, U$1G$1.BANK34_M2@59, U$5.DIR@5
- new net DIR_HALT: R19.1, U$1G$1.BANK34_M1@60, U$8.DIR@5
- new net DIR_IRQ: R4.1, U$1G$2.BANK35_B7@7, U$6.DIR@5
- new net DIR_MPD: R5.1, U$1G$2.BANK35_A7@8, U$4.DIR@5
- new net DIR_RD4: R10.1, U$16.DIR@5, U$1G$2.BANK35_B6@9
- new net DIR_RD5: R13.1, U$14.DIR@5, U$1G$2.BANK35_B5@10
- new net DIR_REF: R20.1, U$1G$2.BANK35_E6@11, U$7.DIR@5
- new net DIR_RST: R21.1, U$17.DIR@5, U$1G$2.BANK35_K5@12
- new net DIR_RW: R22.1, U$1G$2.BANK35_J5@13, U$9.DIR@5
- new net DIR_S4: R23.1, U$12.DIR@5, U$1G$2.BANK35_J4@14
- new net DIR_S5: R24.1, U$11.DIR@5, U$1G$2.BANK35_G5@15
- new net HBUS0: JP3.3, SLOT0.B22, SLOT1.B22, SLOT2.B22, SLOT3.B22, SLOT4.B22, U$1G$2.BANK35_F3@42
- new net HBUS1: JP3.4, SLOT0.B23, SLOT1.B23, SLOT2.B23, SLOT3.B23, SLOT4.B23, U$1G$2.BANK35_F4@41
- new net HBUS2: JP3.5, SLOT0.B24, SLOT1.B24, SLOT2.B24, SLOT3.B24, SLOT4.B24, U$1G$2.BANK35_E1@40
- new net HBUS3: JP3.6, SLOT0.B25, SLOT1.B25, SLOT2.B25, SLOT3.B25, SLOT4.B25, U$1G$2.BANK35_F2@39
- new net HBUS4: JP3.7, SLOT0.B26, SLOT1.B26, SLOT2.B26, SLOT3.B26, SLOT4.B26, U$1G$2.BANK35_E5@38
- new net HBUS5: JP3.8, SLOT0.B27, SLOT1.B27, SLOT2.B27, SLOT3.B27, SLOT4.B27, U$1G$2.BANK35_F5@37
- new net HBUS6: JP3.9, SLOT0.B28, SLOT1.B28, SLOT2.B28, SLOT3.B28, SLOT4.B28, U$1G$2.BANK35_D3@36
- new net HBUS7: JP3.10, SLOT0.B29, SLOT1.B29, SLOT2.B29, SLOT3.B29, SLOT4.B29, U$1G$2.BANK35_E3@35
- new net HBUS8: JP3.11, SLOT0.B30, SLOT1.B30, SLOT2.B30, SLOT3.B30, SLOT4.B30, U$1G$2.BANK35_D1@34
- new net HBUS9: JP3.12, SLOT0.B31, SLOT1.B31, SLOT2.B31, SLOT3.B31, SLOT4.B31, U$1G$2.BANK35_E2@33
- new net HI_A0: CARTRIDGE.A0@5, JP1.16, LVL_ALO.B1@21, U$3.A1
- new net HI_A1: CARTRIDGE.A1@4, JP1.14, LVL_ALO.B2@20, U$3.B1
- new net HI_A10: CARTRIDGE.A10@P, JP1.29, LVL_AHI.B3@19, U$3.A6
- new net HI_A11: CARTRIDGE.A11@N, JP1.27, LVL_AHI.B4@18, U$3.B6
- new net HI_A12: CARTRIDGE.A12@K, JP1.21, LVL_AHI.B5@17, U$3.A7
- new net HI_A13: JP1.41, LVL_AHI.B6@16, U$3.B7
- new net HI_A14: JP1.43, LVL_AHI.B7@15, U$3.A8
- new net HI_A15: JP1.42, LVL_AHI.B8@14, U$3.B8
- new net HI_A2: CARTRIDGE.A2@3, JP1.12, LVL_ALO.B3@19, U$3.A2
- new net HI_A3: CARTRIDGE.A3@2, JP1.10, LVL_ALO.B4@18, U$3.B2
- new net HI_A4: CARTRIDGE.A4@C, JP1.9, LVL_ALO.B5@17, U$3.A3
- new net HI_A5: CARTRIDGE.A5@D, JP1.11, LVL_ALO.B6@16, U$3.B3
- new net HI_A6: CARTRIDGE.A6@E, JP1.13, LVL_ALO.B7@15, U$3.A4
- new net HI_A7: CARTRIDGE.A7@F, JP1.15, LVL_ALO.B8@14, U$3.B4
- new net HI_A8: CARTRIDGE.A8@H, JP1.17, LVL_AHI.B1@21, U$3.A5
- new net HI_A9: CARTRIDGE.A9@J, JP1.19, LVL_AHI.B2@20, U$3.B5
- new net HI_CLK: CARTRIDGE.B02@S, JP1.35, U$15.B@4, U$3.A9
- new net HI_D0: CARTRIDGE.D0@10, JP1.26, LVL_D.B1@21, U$3.B9
- new net HI_D1: CARTRIDGE.D1@9, JP1.24, LVL_D.B2@20, U$3.A10
- new net HI_D2: CARTRIDGE.D2@8, JP1.22, LVL_D.B3@19, U$3.B10
- new net HI_D3: CARTRIDGE.D3@L, JP1.23, LVL_D.B4@18, U$3.A11
- new net HI_D4: CARTRIDGE.D4@6, JP1.18, LVL_D.B5@17, U$3.B11
- new net HI_D5: CARTRIDGE.D5@7, JP1.20, LVL_D.B6@16, U$3.A12
- new net HI_D6: CARTRIDGE.D6@11, JP1.28, LVL_D.B7@15, U$3.B12
- new net HI_D7: CARTRIDGE.D7@M, JP1.25, LVL_D.B8@14, U$3.A13
- new net HI_R/!W!: CARTRIDGE.R/!W!@R, JP1.33, U$3.B17, U$9.B@4
- new net HI_RD4: CARTRIDGE.RD4@A, JP1.7, U$16.B@4, U$3.B15
- new net HI_RD5: CARTRIDGE.RD5@14, JP1.31, U$14.B@4, U$3.A16
- new net LO_A0: LVL_ALO.A1@3, SLOT0.A11, SLOT1.A11, SLOT2.A11, SLOT3.A11, SLOT4.A11, U$1G$1.BANK14_P14@18
- new net LO_A1: LVL_ALO.A2@4, SLOT0.A12, SLOT1.A12, SLOT2.A12, SLOT3.A12, SLOT4.A12, U$1G$1.BANK14_T13@19
- new net LO_A10: LVL_AHI.A3@5, SLOT0.A21, SLOT1.A21, SLOT2.A21, SLOT3.A21, SLOT4.A21, U$1G$1.BANK14_P11@28
- new net LO_A11: LVL_AHI.A4@6, SLOT0.A22, SLOT1.A22, SLOT2.A22, SLOT3.A22, SLOT4.A22, U$1G$1.BANK14_N9@29
- new net LO_A12: LVL_AHI.A5@7, SLOT0.A23, SLOT1.A23, SLOT2.A23, SLOT3.A23, SLOT4.A23, U$1G$1.BANK14_P9@30
- new net LO_A13: LVL_AHI.A6@8, SLOT0.A24, SLOT1.A24, SLOT2.A24, SLOT3.A24, SLOT4.A24, U$1G$1.BANK14_T10@31
- new net LO_A14: LVL_AHI.A7@9, SLOT0.A25, SLOT1.A25, SLOT2.A25, SLOT3.A25, SLOT4.A25, U$1G$1.BANK14_R11@32
- new net LO_A15: LVL_AHI.A8@10, SLOT0.A26, SLOT1.A26, SLOT2.A26, SLOT3.A26, SLOT4.A26, U$1G$1.BANK14_T9@33
- new net LO_A2: LVL_ALO.A3@5, SLOT0.A13, SLOT1.A13, SLOT2.A13, SLOT3.A13, SLOT4.A13, U$1G$1.BANK14_R13@20
- new net LO_A3: LVL_ALO.A4@6, SLOT0.A14, SLOT1.A14, SLOT2.A14, SLOT3.A14, SLOT4.A14, U$1G$1.BANK14_T12@21
- new net LO_A4: LVL_ALO.A5@7, SLOT0.A15, SLOT1.A15, SLOT2.A15, SLOT3.A15, SLOT4.A15, U$1G$1.BANK14_R12@22
- new net LO_A5: LVL_ALO.A6@8, SLOT0.A16, SLOT1.A16, SLOT2.A16, SLOT3.A16, SLOT4.A16, U$1G$1.BANK14_L13@23
- new net LO_A6: LVL_ALO.A7@9, SLOT0.A17, SLOT1.A17, SLOT2.A17, SLOT3.A17, SLOT4.A17, U$1G$1.BANK14_N12@24
- new net LO_A7: LVL_ALO.A8@10, SLOT0.A18, SLOT1.A18, SLOT2.A18, SLOT3.A18, SLOT4.A18, U$1G$1.BANK14_K12@25
- new net LO_A8: LVL_AHI.A1@3, SLOT0.A19, SLOT1.A19, SLOT2.A19, SLOT3.A19, SLOT4.A19, U$1G$1.BANK14_K13@26
- new net LO_A9: LVL_AHI.A2@4, SLOT0.A20, SLOT1.A20, SLOT2.A20, SLOT3.A20, SLOT4.A20, U$1G$1.BANK14_P10@27
- new net LO_CLK: SLOT0.A28, SLOT1.A28, SLOT2.A28, SLOT3.A28, SLOT4.A28, U$15.A@3, U$1G$1.BANK14_T8@35
- new net LO_D0: LVL_D.A1@3, SLOT0.B7, SLOT1.B7, SLOT2.B7, SLOT3.B7, SLOT4.B7, U$1G$1.BANK14_R8@36
- new net LO_D1: LVL_D.A2@4, SLOT0.B8, SLOT1.B8, SLOT2.B8, SLOT3.B8, SLOT4.B8, U$1G$1.BANK14_T7@37
- new net LO_D2: LVL_D.A3@5, SLOT0.B9, SLOT1.B9, SLOT2.B9, SLOT3.B9, SLOT4.B9, U$1G$1.BANK14_R7@38
- new net LO_D3: LVL_D.A4@6, SLOT0.B10, SLOT1.B10, SLOT2.B10, SLOT3.B10, SLOT4.B10, U$1G$1.BANK14_T5@39
- new net LO_D4: LVL_D.A5@7, SLOT0.B11, SLOT1.B11, SLOT2.B11, SLOT3.B11, SLOT4.B11, U$1G$1.BANK14_R6@40
- new net LO_D5: LVL_D.A6@8, SLOT0.B12, SLOT1.B12, SLOT2.B12, SLOT3.B12, SLOT4.B12, U$1G$1.BANK14_P6@41
- new net LO_D6: LVL_D.A7@9, SLOT0.B13, SLOT1.B13, SLOT2.B13, SLOT3.B13, SLOT4.B13, U$1G$1.BANK14_R5@42
- new net LO_D7: LVL_D.A8@10, SLOT0.B14, SLOT1.B14, SLOT2.B14, SLOT3.B14, SLOT4.B14, U$1G$1.BANK14_N6@43
- new net LO_R/!W!: SLOT0.B19, SLOT1.B19, SLOT2.B19, SLOT3.B19, SLOT4.B19, U$1G$1.BANK34_R1@52, U$9.A@3
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Other:
- note added: "+5V Card-present Slot ID GND"
- note added: "B1,2,3 B4 A1,2,3 A4,5,6,7"
- note added: "FPGA"
- note added: "High voltage signals"
- note added: "Level changers"
- note added: "Place pull-ups close to card socket"
- note added: "Serial & Config"
- note added: "Top 7 SD card Next 4 RS232 Next 34 Bus"
- note added: "Video Out"
- note removed: "@48"
- note removed: "Board config"
- note removed: "Cartridge support"
- note removed: "Debugging LEDs"
- note removed: "HOST_DIR0 :"
- note removed: "Host data bus"
- note removed: "LCDT"
- note removed: "Serial IO / Slot presence"
- note removed: "Slot id: 1,0,0"
- note removed: "XIO POWER"

Commit message: - Add a +5v plane to cover where useful - Have a better placement of the HBUS extension - Gives at least 10cm of space for cards
Parts:
- removed C10, C61, C62, C64, C66, C69, C7, C70: 0.1uF, rcl:C-EUC0201
- removed R1, R20, R23, R24: 10K, rcl:R-EU_R0201
- removed U$11, U$12, U$13, U$7: 74LVC1T45GWSOT866, sjg-logic:74LVC1T45GWSOT866
- JP3: device pinhead:PINHD-2X8 -> pinhead:PINHD-2X10
Connections:
- removed net !HI_REF!: JP1.40, U$3.B16, U$7.B@4
- removed net !LO_S4!: SLOT0.B20, SLOT1.B20, SLOT2.B20, SLOT3.B20, SLOT4.B20, U$12.A@3, U$1G$1.BANK34_M5@53
- removed net !LO_S5!: SLOT0.B21, SLOT1.B21, SLOT2.B21, SLOT3.B21, SLOT4.B21, U$11.A@3, U$1G$1.BANK34_N4@54
- new net HBUS10: JP3.13, SLOT0.B28, SLOT1.B28, SLOT2.B28, SLOT3.B28, SLOT4.B28, U$1G$1.BANK34_R2@51
- new net HBUS11: JP3.14, SLOT0.B29, SLOT1.B29, SLOT2.B29, SLOT3.B29, SLOT4.B29, U$1G$1.BANK34_R1@52
- new net HBUS12: JP3.15, SLOT0.B30, SLOT1.B30, SLOT2.B30, SLOT3.B30, SLOT4.B30, U$1G$1.BANK34_M5@53
- new net HBUS13: JP3.16, SLOT0.B31, SLOT1.B31, SLOT2.B31, SLOT3.B31, SLOT4.B31, U$1G$1.BANK34_N4@54
- net !HI_CCTL!: no longer U$13.B@4
- net !HI_S4!: now also JP1.40, U$3.B16; no longer U$12.B@4
- net !HI_S5!: now also JP1.44, U$3.B18; no longer U$11.B@4
- net !LO_CCTL!: no longer U$13.A@3, U$1G$1.BANK14_R10@34
- net !LO_EXTSEL!: now also U$1G$1.BANK14_N6@43; no longer U$1G$1.BANK14_M6@44
- net !LO_HALT!: now also SLOT0.B13, SLOT1.B13, SLOT2.B13, SLOT3.B13, SLOT4.B13, U$1G$1.BANK14_M6@44; no longer SLOT0.A30, SLOT1.A30, SLOT2.A30, SLOT3.A30, SLOT4.A30, U$1G$1.BANK34_L5@45
- net !LO_IRQ!: now also SLOT0.B14, SLOT1.B14, SLOT2.B14, SLOT3.B14, SLOT4.B14, U$1G$1.BANK34_L5@45; no longer SLOT0.A31, SLOT1.A31, SLOT2.A31, SLOT3.A31, SLOT4.A31, U$1G$1.BANK34_P5@46
- net !LO_MPD!: now also SLOT0.A30, SLOT1.A30, SLOT2.A30, SLOT3.A30, SLOT4.A30, U$1G$1.BANK34_P5@46; no longer SLOT0.A32, SLOT1.A32, SLOT2.A32, SLOT3.A32, SLOT4.A32, U$1G$1.BANK34_T4@47
- net !LO_REF!: now also SLOT0.B15, SLOT1.B15, SLOT2.B15, SLOT3.B15, SLOT4.B15; no longer SLOT0.B17, SLOT1.B17, SLOT2.B17, SLOT3.B17, SLOT4.B17, U$1G$1.BANK34_T2@50, U$7.A@3
- net !LO_RST!: now also SLOT0.B16, SLOT1.B16, SLOT2.B16, SLOT3.B16, SLOT4.B16, U$1G$1.BANK34_R3@49; no longer SLOT0.B18, SLOT1.B18, SLOT2.B18, SLOT3.B18, SLOT4.B18, U$1G$1.BANK34_R2@51
- net +3V3: no longer C61.1, C62.1, C64.1, C7.1, U$11.VCCA@1, U$12.VCCA@1, U$13.VCCA@1, U$7.VCCA@1
- net +5V: no longer C10.1, C66.1, C69.1, C70.1, U$11.VCCB@6, U$12.VCCB@6, U$13.VCCB@6, U$7.VCCB@6
- net DIR_CCTL: no longer R1.1, U$13.DIR@5
- net DIR_REF: no longer R20.1, U$7.DIR@5
- net DIR_S4: no longer R23.1, U$12.DIR@5
- net DIR_S5: no longer R24.1, U$11.DIR@5
- net GND: now also JP3.17, JP3.18, JP3.19, JP3.20, SLOT0.B32, SLOT1.B32, SLOT2.B32, SLOT3.B32, SLOT4.B32; no longer C10.2, C61.2, C62.2, C64.2, C66.2, C69.2, C7.2, C70.2, JP1.44, JP3.13, JP3.14, JP3.15, JP3.16, R1.2, R20.2, R23.2, R24.2, SLOT0.A6, SLOT0.A7, SLOT1.A6, SLOT1.A7, SLOT2.A6, SLOT2.A7, SLOT3.A6, SLOT3.A7, SLOT4.A6, U$11.GND@2, U$12.GND@2, U$13.GND@2, U$7.GND@2
- net HBUS0: now also SLOT0.B18, SLOT1.B18, SLOT2.B18, SLOT3.B18, SLOT4.B18; no longer SLOT0.B22, SLOT1.B22, SLOT2.B22, SLOT3.B22, SLOT4.B22
- net HBUS1: now also SLOT0.B19, SLOT1.B19, SLOT2.B19, SLOT3.B19, SLOT4.B19; no longer SLOT0.B23, SLOT1.B23, SLOT2.B23, SLOT3.B23, SLOT4.B23
- net HBUS2: now also SLOT0.B20, SLOT1.B20, SLOT2.B20, SLOT3.B20, SLOT4.B20; no longer SLOT0.B24, SLOT1.B24, SLOT2.B24, SLOT3.B24, SLOT4.B24
- net HBUS3: now also SLOT0.B21, SLOT1.B21, SLOT2.B21, SLOT3.B21, SLOT4.B21; no longer SLOT0.B25, SLOT1.B25, SLOT2.B25, SLOT3.B25, SLOT4.B25
- net HBUS4: now also SLOT0.B22, SLOT1.B22, SLOT2.B22, SLOT3.B22, SLOT4.B22; no longer SLOT0.B26, SLOT1.B26, SLOT2.B26, SLOT3.B26, SLOT4.B26
- net HBUS5: now also SLOT0.B23, SLOT1.B23, SLOT2.B23, SLOT3.B23, SLOT4.B23; no longer SLOT0.B27, SLOT1.B27, SLOT2.B27, SLOT3.B27, SLOT4.B27
- net HBUS6: now also SLOT0.B24, SLOT1.B24, SLOT2.B24, SLOT3.B24, SLOT4.B24; no longer SLOT0.B28, SLOT1.B28, SLOT2.B28, SLOT3.B28, SLOT4.B28
- net HBUS7: now also SLOT0.B25, SLOT1.B25, SLOT2.B25, SLOT3.B25, SLOT4.B25; no longer SLOT0.B29, SLOT1.B29, SLOT2.B29, SLOT3.B29, SLOT4.B29
- net HBUS8: now also SLOT0.B26, SLOT1.B26, SLOT2.B26, SLOT3.B26, SLOT4.B26; no longer SLOT0.B30, SLOT1.B30, SLOT2.B30, SLOT3.B30, SLOT4.B30
- net HBUS9: now also SLOT0.B27, SLOT1.B27, SLOT2.B27, SLOT3.B27, SLOT4.B27; no longer SLOT0.B31, SLOT1.B31, SLOT2.B31, SLOT3.B31, SLOT4.B31
- net LO_CLK: now also U$1G$1.BANK14_R10@34; no longer U$1G$1.BANK14_T8@35
- net LO_D0: now also SLOT0.B5, SLOT1.B5, SLOT2.B5, SLOT3.B5, SLOT4.B5, U$1G$1.BANK14_T8@35; no longer SLOT0.B7, SLOT1.B7, SLOT2.B7, SLOT3.B7, SLOT4.B7, U$1G$1.BANK14_R8@36
- net LO_D1: now also SLOT0.B6, SLOT1.B6, SLOT2.B6, SLOT3.B6, SLOT4.B6, U$1G$1.BANK14_R8@36; no longer SLOT0.B8, SLOT1.B8, SLOT2.B8, SLOT3.B8, SLOT4.B8, U$1G$1.BANK14_T7@37
- net LO_D2: now also SLOT0.B7, SLOT1.B7, SLOT2.B7, SLOT3.B7, SLOT4.B7, U$1G$1.BANK14_T7@37; no longer SLOT0.B9, SLOT1.B9, SLOT2.B9, SLOT3.B9, SLOT4.B9, U$1G$1.BANK14_R7@38
- net LO_D3: now also SLOT0.B8, SLOT1.B8, SLOT2.B8, SLOT3.B8, SLOT4.B8, U$1G$1.BANK14_R7@38; no longer SLOT0.B10, SLOT1.B10, SLOT2.B10, SLOT3.B10, SLOT4.B10, U$1G$1.BANK14_T5@39
- net LO_D4: now also SLOT0.B9, SLOT1.B9, SLOT2.B9, SLOT3.B9, SLOT4.B9, U$1G$1.BANK14_T5@39; no longer SLOT0.B11, SLOT1.B11, SLOT2.B11, SLOT3.B11, SLOT4.B11, U$1G$1.BANK14_R6@40
- net LO_D5: now also SLOT0.B10, SLOT1.B10, SLOT2.B10, SLOT3.B10, SLOT4.B10, U$1G$1.BANK14_R6@40; no longer SLOT0.B12, SLOT1.B12, SLOT2.B12, SLOT3.B12, SLOT4.B12, U$1G$1.BANK14_P6@41
- net LO_D6: now also SLOT0.B11, SLOT1.B11, SLOT2.B11, SLOT3.B11, SLOT4.B11, U$1G$1.BANK14_P6@41; no longer SLOT0.B13, SLOT1.B13, SLOT2.B13, SLOT3.B13, SLOT4.B13, U$1G$1.BANK14_R5@42
- net LO_D7: now also SLOT0.B12, SLOT1.B12, SLOT2.B12, SLOT3.B12, SLOT4.B12, U$1G$1.BANK14_R5@42; no longer SLOT0.B14, SLOT1.B14, SLOT2.B14, SLOT3.B14, SLOT4.B14, U$1G$1.BANK14_N6@43
- net LO_R/!W!: now also SLOT0.B17, SLOT1.B17, SLOT2.B17, SLOT3.B17, SLOT4.B17, U$1G$1.BANK34_T2@50; no longer SLOT0.B19, SLOT1.B19, SLOT2.B19, SLOT3.B19, SLOT4.B19, U$1G$1.BANK34_R1@52
- net LO_RD4: now also SLOT0.A31, SLOT1.A31, SLOT2.A31, SLOT3.A31, SLOT4.A31, U$1G$1.BANK34_T4@47; no longer SLOT0.B15, SLOT1.B15, SLOT2.B15, SLOT3.B15, SLOT4.B15, U$1G$1.BANK34_T3@48
- net LO_RD5: now also SLOT0.A32, SLOT1.A32, SLOT2.A32, SLOT3.A32, SLOT4.A32, U$1G$1.BANK34_T3@48; no longer SLOT0.B16, SLOT1.B16, SLOT2.B16, SLOT3.B16, SLOT4.B16, U$1G$1.BANK34_R3@49
- net VALID_RD: now also SLOT0.A7, SLOT1.A7, SLOT2.A7, SLOT3.A7, SLOT4.A7; no longer SLOT0.B5, SLOT1.B5, SLOT2.B5, SLOT3.B5, SLOT4.B5
- net VALID_WR: now also SLOT0.A6, SLOT1.A6, SLOT2.A6, SLOT3.A6, SLOT4.A6; no longer SLOT0.B6, SLOT1.B6, SLOT2.B6, SLOT3.B6, SLOT4.B6
Other:
- note added: "Make pinout same as MiniPBI+ (XLD)"
- moved on the sheet: C11, C12, C53, C54, C55, C56, C63, C65, C68, C71, C72, LD_0P1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
