File: boards/xio4/xio4.brd (EAGLE design)
At the start: 170 x 170 mm, 95 parts

Commit message: Start looking at the mezzanine board
Parts:
- added JP2: (no value), pinhead-2:2X15SMD
- JP1: device pinhead:2X25 -> pinhead-2:2X15SMD
- moved ARCH_ID 159.4 mm to (164.1, 61.7), turned to 270 degrees
- moved MEM_ID 159.1 mm to (164.1, 82.0), turned to 270 degrees
- moved PID 158.0 mm to (164.1, 73.2), turned to 270 degrees
- moved R6 148.1 mm to (157.7, 57.9), turned to 180 degrees
- moved R7 147.2 mm to (157.7, 60.5), turned to 180 degrees
- moved R18 146.9 mm to (157.7, 83.3), turned to 180 degrees
- moved R8 146.5 mm to (157.7, 63.0), turned to 180 degrees
- moved R17 146.2 mm to (157.7, 80.8), turned to 180 degrees
- moved R123 146.0 mm to (157.7, 79.5), turned to 0 degrees
- moved R9 145.9 mm to (157.7, 65.5), turned to 180 degrees
- moved R122 145.7 mm to (157.7, 66.8), turned to 0 degrees
- moved R124 145.5 mm to (157.7, 77.0), turned to 0 degrees
- moved R16 145.4 mm to (157.7, 75.7), turned to 180 degrees
- moved R14 145.3 mm to (157.7, 70.6), turned to 180 degrees
- moved R15 145.3 mm to (157.7, 73.2), turned to 180 degrees
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Connections:
- net !HI_CCTL!: no longer JP1.34
- net !HI_EXTSEL!: no longer JP1.36
- net !HI_HALT!: no longer JP1.39
- net !HI_IRQ!: no longer JP1.37
- net !HI_MPD!: no longer JP1.38
- net !HI_RST!: no longer JP1.32
- net !HI_S4!: no longer JP1.40, JP1.8
- net !HI_S5!: no longer JP1.30, JP1.44
- net +5V: no longer JP1.1, JP1.2, JP1.3, JP1.4, JP1.5, JP1.6
- net GND: no longer JP1.45, JP1.46, JP1.47, JP1.48, JP1.49, JP1.50
- net HI_A0: no longer JP1.16
- net HI_A1: no longer JP1.14
- net HI_A10: no longer JP1.29
- net HI_A11: no longer JP1.27
- net HI_A12: no longer JP1.21
- net HI_A13: no longer JP1.41
- net HI_A14: no longer JP1.43
- net HI_A15: no longer JP1.42
- net HI_A2: no longer JP1.12
- net HI_A3: no longer JP1.10
- net HI_A4: no longer JP1.9
- net HI_A5: no longer JP1.11
- net HI_A6: no longer JP1.13
- net HI_A7: no longer JP1.15
- net HI_A8: no longer JP1.17
- net HI_A9: no longer JP1.19
- net HI_CLK: no longer JP1.35
- net HI_D0: no longer JP1.26
- net HI_D1: no longer JP1.24
- net HI_D2: no longer JP1.22
- net HI_D3: no longer JP1.23
- net HI_D4: no longer JP1.18
- net HI_D5: no longer JP1.20
- net HI_D6: no longer JP1.28
- net HI_D7: no longer JP1.25
- net HI_R/!W!: no longer JP1.33
- net HI_RD4: no longer JP1.7
- net HI_RD5: no longer JP1.31
Other:
- board text added: "Top board - Zturn Lite Middle - B2B, Cartridge, SAS & HDMI underneath Base - PCIe x5, Dips All SMT parts are 1206"
- board text removed: "Top board - Zturn Lite Middle - B2B, SAS & HDMI underneath Base - Cartridge, MPBI+, PCIe x5, Dips All SMT parts are 1206"
