File: boards/xio5/xio5.brd (EAGLE design)
At the start: 170 x 170 mm, 94 parts, among them IC1 SN74LVC138APWR, IC2 XRA1405IL24-F, J1 98424-G52-14ALF, X1 1365-80, X2 1365-80

Commit message: Routed at 4/4
Parts:
- removed JP1: (no value), pinhead:1X07
- removed JP2: (no value), pinhead-2:2X20M
- removed JP3: (no value), pinhead-2:2X10M
- removed JP5: (no value), pinhead-2:2X04M
- removed R10, R13, R2: 10K, rcl:R0201
- removed X1, X2: 1365-80, con-leotronics:1365-80
- added AUDIO_CONN: (no value), pinhead-2:2X06M
- added AUX_JTAG: (no value), pinhead:1X07
- added BOARD_POWER: 1706714, samacsys:1706714
- added INTERNAL_EXP: (no value), pinhead-2:2X16M
- added R11, R12, R14, R18, R20, R7, R8, R9: 10K, rcl:R0201
- added SPI7_CONN: (no value), pinhead-2:2X04M
- added SW_CONFIG: (no value), SparkFun:DIPSWITCH-08
- moved C16 6.48 mm to (138.9, 143.6)
- moved C13 6.48 mm to (133.8, 129.6)
- moved C18 6.48 mm to (139.2, 129.3)
- moved LVL_AHI 6.48 mm to (136.4, 138.5)
- moved R25 6.48 mm to (132.6, 129.6)
- moved C15 6.48 mm to (137.7, 115.7)
- moved C3 6.48 mm to (133.8, 115.7)
- moved LVL_ALO 6.48 mm to (136.4, 110.6)
- moved LVL_D 6.48 mm to (136.4, 124.6)
- moved C17 6.48 mm to (133.8, 143.6)
- moved R26 6.48 mm to (132.6, 143.6)
- renumbered JP4 to SPI6_CONN
Connections:
- removed net DIR_CLK: R2.1
- removed net DIR_RD4: R10.1
- removed net DIR_RD5: R13.1
- removed net XBUS0: JP2.26, JP3.13, ZTURN.CN2_28
- removed net XBUS1: JP2.28, JP3.15, ZTURN.CN2_32
- removed net XBUS2: JP2.30, JP3.17, ZTURN.CN2_34
- removed net XBUS3: JP2.32, JP3.19, ZTURN.CN2_36
- removed net XBUS4: JP2.34, ZTURN.CN2_38
- removed net XBUS5: JP2.36, ZTURN.CN2_42
- removed net XBUS6: JP2.38, ZTURN.CN2_44
- removed net XBUS7: JP2.40, ZTURN.CN2_46
- removed net XBUS8: ZTURN.CN2_48
- new net !HDMI_INT!: ZTURN.CN1_77, ZTURN.CN2_28
- new net CFG0: IC2.1, R14.1, SW_CONFIG.1
- new net CFG1: IC2.2, R12.1, SW_CONFIG.2
- new net CFG2: IC2.3, R11.1, SW_CONFIG.3
- new net CFG3: IC2.4, R9.1, SW_CONFIG.4
- new net CFG4: IC2.5, R8.1, SW_CONFIG.5
- new net CFG5: IC2.6, R7.1, SW_CONFIG.6
- new net CFG6: IC2.7, R18.1, SW_CONFIG.7
- new net CFG7: IC2.8, R20.1, SW_CONFIG.8
- net !SRST!: now also AUX_JTAG.6; no longer JP1.6
- net +3V3: now also AUDIO_CONN.7, AUX_JTAG.1, INTERNAL_EXP.6, INTERNAL_EXP.8, R11.2, R12.2, R14.2, R18.2, R20.2, R7.2, R8.2, R9.2; no longer JP1.1, JP2.6, JP2.8, JP3.5, JP3.7
- net +5V: now also AUDIO_CONN.5, BOARD_POWER.1, BOARD_POWER.2, INTERNAL_EXP.2, INTERNAL_EXP.4, SPI7_CONN.1; no longer JP2.2, JP2.4, JP3.1, JP3.3, JP5.1
- net GND: now also AUDIO_CONN.11, AUDIO_CONN.4, AUDIO_CONN.9, AUX_JTAG.7, INTERNAL_EXP.30, INTERNAL_EXP.32, SPI7_CONN.8, SW_CONFIG.10, SW_CONFIG.11, SW_CONFIG.12, SW_CONFIG.13, SW_CONFIG.14, SW_CONFIG.15, SW_CONFIG.16, SW_CONFIG.9; no longer JP1.7, JP2.24, JP2.33, JP2.39, JP3.11, JP3.20, JP3.6, JP3.8, JP3.9, JP5.7, JP5.8, R10.2, R13.2, R2.2, SPI6_CONN.7
- net I2C0_SCL: now also AUDIO_CONN.1, INTERNAL_EXP.26; no longer JP2.37, JP3.4
- net I2C0_SDA: now also AUDIO_CONN.3, INTERNAL_EXP.24; no longer JP2.35, JP3.2
- net N$2: now also AUDIO_CONN.2; no longer JP3.10
- net N$6: now also AUDIO_CONN.12, ZTURN.CN1_72; no longer JP3.12, ZTURN.CN1_75
- net N$7: now also AUDIO_CONN.10, ZTURN.CN1_74; no longer JP3.14, ZTURN.CN1_73
- net N$8: now also AUDIO_CONN.8, ZTURN.CN1_73; no longer JP3.16, ZTURN.CN1_74
- net N$9: now also AUDIO_CONN.6, ZTURN.CN1_75; no longer JP3.18, ZTURN.CN1_72
- net S5_PRESENT: now also INTERNAL_EXP.20; no longer JP2.20
- net S7_PRESENT: now also SPI7_CONN.5; no longer JP5.5
- net SPI1_CLK: now also SPI7_CONN.2; no longer JP5.2
- net SPI1_MISO: now also SPI7_CONN.4; no longer JP5.4
- net SPI1_MOSI: now also SPI7_CONN.6; no longer JP5.6
- net SPI2_CLK: now also INTERNAL_EXP.10; no longer JP2.10
- net SPI2_CS1: now also INTERNAL_EXP.12; no longer JP2.12
- net SPI2_IRQ: now also INTERNAL_EXP.16; no longer JP2.16
- net SPI2_MISO: now also INTERNAL_EXP.14; no longer JP2.14
- net SPI2_MOSI: now also INTERNAL_EXP.18; no longer JP2.18
- net SPI_IRQ0: now also ZTURN.CN2_48; no longer IC2.1
- net SPI_IRQ1: now also ZTURN.CN2_46; no longer IC2.2
- net SPI_IRQ2: now also ZTURN.CN2_44; no longer IC2.3
- net SPI_IRQ3: now also ZTURN.CN2_42; no longer IC2.4
- net SPI_IRQ4: now also ZTURN.CN2_38; no longer IC2.5
- net SPI_IRQ5: now also INTERNAL_EXP.22, ZTURN.CN2_36; no longer IC2.6, JP2.22
- net SPI_IRQ6: now also ZTURN.CN2_34; no longer IC2.7
- net SPI_IRQ7: now also SPI7_CONN.3, ZTURN.CN2_32; no longer IC2.8, JP5.3
- net SPI_SS5: now also INTERNAL_EXP.28
- net SPI_SS6: now also SPI6_CONN.7
- net SPI_SS7: now also SPI7_CONN.7
- net TCK: now also AUX_JTAG.3; no longer JP1.3
- net TDI: now also AUX_JTAG.5; no longer JP1.5
- net TDO: now also AUX_JTAG.4; no longer JP1.4
- net TMS: now also AUX_JTAG.2; no longer JP1.2
- net ZBUS0: now also INTERNAL_EXP.31; no longer JP2.31
- net ZBUS1: now also INTERNAL_EXP.29; no longer JP2.29
- net ZBUS10: now also INTERNAL_EXP.11; no longer JP2.11
- net ZBUS11: now also INTERNAL_EXP.9; no longer JP2.9
- net ZBUS12: now also INTERNAL_EXP.7; no longer JP2.7
- net ZBUS13: now also INTERNAL_EXP.5; no longer JP2.5
- net ZBUS14: now also INTERNAL_EXP.3; no longer JP2.3
- net ZBUS15: now also INTERNAL_EXP.1; no longer JP2.1
- net ZBUS2: now also INTERNAL_EXP.27; no longer JP2.27
- net ZBUS3: now also INTERNAL_EXP.25; no longer JP2.25
- net ZBUS4: now also INTERNAL_EXP.23; no longer JP2.23
- net ZBUS5: now also INTERNAL_EXP.21; no longer JP2.21
- net ZBUS6: now also INTERNAL_EXP.19; no longer JP2.19
- net ZBUS7: now also INTERNAL_EXP.17; no longer JP2.17
- net ZBUS8: now also INTERNAL_EXP.15; no longer JP2.15
- net ZBUS9: now also INTERNAL_EXP.13; no longer JP2.13
Routing:
- net CFG2: track 0.00 -> 178.8 mm, vias 0 -> 1
- net CFG6: track 0.00 -> 177.2 mm, vias 0 -> 1
- net CFG5: track 0.00 -> 169.5 mm, vias 0 -> 1
- net CFG4: track 0.00 -> 169.2 mm, vias 0 -> 1
- net CFG3: track 0.00 -> 168.9 mm, vias 0 -> 1
- net CFG0: track 0.00 -> 160.2 mm, vias 0 -> 3
- net CFG7: track 0.00 -> 145.0 mm, vias 0 -> 2
- net CFG1: track 0.00 -> 134.0 mm, vias 0 -> 1
- net XBUS1: track 120.1 -> 0.00 mm
- net XBUS3: track 105.9 -> 0.00 mm, vias 3 -> 0
- net SPI_SS7: track 0.00 -> 104.8 mm, vias 0 -> 1
- net XBUS0: track 102.0 -> 0.00 mm, vias 1 -> 0
- net XBUS2: track 100.2 -> 0.00 mm, vias 2 -> 0
- net SPI_SS6: track 0.00 -> 85.3 mm
- net GND: track 703.2 -> 621.8 mm, vias 21 -> 15
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