File: boards/xio6/xio.sch (EAGLE design)
At the start: 35 parts, among them IC1 STM32MP157AAA3, IC2 IS43TR16256AL-125KBL, IC3 TFP410PAP, IC4 STPMIC1APQR, J1 DC-005, J3 RJMG2310228A0ER

Commit message: Get the smaller PCIe slots organised
Parts:
- removed C54: 0.1uF, rcl:C-EUC0201
- removed EXP0, EXP1, EXP4: 10018784-10210TLF, samacsys:10018784-10210TLF
- removed JP2: (no value), pinhead-2:PINHD-2X20_2.00
- removed LD_0P1, LD_1P, LD_2P, LD_3P, LD_4P: SML-D12D1WT86, led:LEDCHIPLED_0603
- added C1: 0.1uF, rcl:C-EUC0201
- added LD0, LD1, LD2, LD3, LD4: SML-D12D1WT86, led:LEDCHIPLED_0603
- added R1, R2, R3, R4, R5: 10K, rcl:R-EU_R0201
- added SLOT0, SLOT1, SLOT4: 10018784-10210TLF, samacsys:10018784-10210TLF
- added U1: USD-SOCKETNEW, SparkFun:USD-SOCKETNEW
- renumbered EXP2 to SLOT2, EXP3 to SLOT3
Connections:
- net !HI_CCTL! renamed !CCTL!
- net !HI_EXTSEL! renamed !EXTSEL!
- net !HI_HALT! renamed !HALT!
- net !HI_IRQ! renamed !IRQ!
- net !HI_MPD! renamed !MPD!
- net !HI_RST! renamed !RST!
- net !HI_S4! renamed !S4!
- net !HI_S5! renamed !S5!
- net HI_CLK renamed CLK
- net HI_R/!W! renamed R/!W!
- net HI_RD4 renamed RD4
- net HI_RD5 renamed RD5
- removed net !LO_EXTSEL!: EXP0.B11, EXP1.B11, EXP4.B11, SLOT2.B11, SLOT3.B11
- removed net !LO_MPD!: EXP0.B13, EXP1.B13, EXP4.B13, SLOT2.B13, SLOT3.B13
- removed net !LO_RST!: EXP0.B7, EXP1.B7, EXP4.B7, SLOT2.B7, SLOT3.B7
- removed net HI_A0: U$1.A0@16, U$3.A1
- removed net HI_A1: U$1.A1@14, U$3.B1
- removed net HI_A10: U$1.A10@46, U$3.A6
- removed net HI_A11: U$1.A11@44, U$3.B6
- removed net HI_A12: U$1.A12@42, U$3.A7
- removed net HI_A13: U$1.A13@40, U$3.B7
- removed net HI_A14: U$1.A14@38, U$3.A8
- removed net HI_A15: U$1.A15@36, U$3.B8
- removed net HI_A2: U$1.A2@12, U$3.A2
- removed net HI_A3: U$1.A3@10, U$3.B2
- removed net HI_A4: U$1.A4@8, U$3.A3
- removed net HI_A5: U$1.A5@6, U$3.B3
- removed net HI_A6: U$1.A6@4, U$3.A4
- removed net HI_A7: U$1.A7@2, U$3.B4
- removed net HI_A8: U$1.A8@50, U$3.A5
- removed net HI_A9: U$1.A9@48, U$3.B5
- removed net HI_D0: U$1.D0@15, U$3.B9
- removed net HI_D1: U$1.D1@13, U$3.A10
- removed net HI_D2: U$1.D2@11, U$3.B10
- removed net HI_D3: U$1.D3@9, U$3.A11
- removed net HI_D4: U$1.D4@7, U$3.B11
- removed net HI_D5: U$1.D5@5, U$3.A12
- removed net HI_D6: U$1.D6@3, U$3.B12
- removed net HI_D7: U$1.D7@1, U$3.A13
- removed net I2C0_SCL: JP2.37
- removed net I2C0_SDA: JP2.35
- removed net LO_A10: EXP0.A13, EXP1.A13, EXP4.A13, SLOT2.A13, SLOT3.A13
- removed net LO_A11: EXP0.A15, EXP1.A15, EXP4.A15, SLOT2.A15, SLOT3.A15
- removed net LO_A12: EXP0.A17, EXP1.A17, EXP4.A17, SLOT2.A17, SLOT3.A17
- removed net LO_A13: EXP0.B1, EXP1.B1, EXP4.B1, SLOT2.B1, SLOT3.B1
- removed net LO_A14: EXP0.B3, EXP1.B3, EXP4.B3, SLOT2.B3, SLOT3.B3
- removed net LO_A15: EXP0.B5, EXP1.B5, EXP4.B5, SLOT2.B5, SLOT3.B5
- removed net LO_A4: EXP0.A1, EXP1.A1, EXP4.A1, SLOT2.A1, SLOT3.A1
- removed net LO_A5: EXP0.A3, EXP1.A3, EXP4.A3, SLOT2.A3, SLOT3.A3
- removed net LO_A6: EXP0.A5, EXP1.A5, EXP4.A5, SLOT2.A5, SLOT3.A5
- removed net LO_A7: EXP0.A7, EXP1.A7, EXP4.A7, SLOT2.A7, SLOT3.A7
- removed net LO_A8: EXP0.A9, EXP1.A9, EXP4.A9, SLOT2.A9, SLOT3.A9
- removed net LO_A9: EXP0.A11, EXP1.A11, EXP4.A11, SLOT2.A11, SLOT3.A11
- removed net LO_CLK: EXP0.B9, EXP1.B9, EXP4.B9, SLOT2.B9, SLOT3.B9
- removed net LO_R/!W!: EXP0.A2, EXP1.A2, EXP4.A2, SLOT2.A2, SLOT3.A2
- removed net LO_RD4: EXP0.B15, EXP1.B15, EXP4.B15, SLOT2.B15, SLOT3.B15
- removed net LO_RD5: EXP0.B17, EXP1.B17, EXP4.B17, SLOT2.B17, SLOT3.B17
- removed net N$101: LD_4P.A, R107.2
- removed net N$91: LD_1P.A, R98.2
- removed net N$94: LD_2P.A, R101.2
- removed net N$97: LD_3P.A, R104.2
- removed net S0_PRESENT: R27.1, R61.2
- removed net S1_PRESENT: R62.2, R98.1
- removed net S2_PRESENT: R101.1, R63.2
- removed net S3_PRESENT: R104.1, R64.2
- removed net S4_PRESENT: R107.1, R65.2
- removed net S5_PRESENT: JP2.20
- removed net SPI2_CS1: JP2.12
- removed net SPI2_IRQ: JP2.16
- removed net SPI_IRQ5: JP2.22
- removed net XBUS0: JP2.26
- removed net XBUS1: JP2.28
- removed net XBUS2: JP2.30
- removed net XBUS3: JP2.32
- removed net XBUS4: JP2.34
- removed net XBUS5: JP2.36
- removed net XBUS6: JP2.38
- removed net XBUS7: JP2.40
- removed net ZBUS0: EXP0.A4, EXP1.A4, EXP4.A4, JP2.31, SLOT2.A4, SLOT3.A4
- removed net ZBUS1: EXP0.A6, EXP1.A6, EXP4.A6, JP2.29, SLOT2.A6, SLOT3.A6
- removed net ZBUS10: EXP0.B6, EXP1.B6, EXP4.B6, JP2.11, SLOT2.B6, SLOT3.B6
- removed net ZBUS11: EXP0.B8, EXP1.B8, EXP4.B8, JP2.9, SLOT2.B8, SLOT3.B8
- removed net ZBUS12: EXP0.B10, EXP1.B10, EXP4.B10, JP2.7, SLOT2.B10, SLOT3.B10
- removed net ZBUS13: EXP0.B12, EXP1.B12, EXP4.B12, JP2.5, SLOT2.B12, SLOT3.B12
- removed net ZBUS14: EXP0.B14, EXP1.B14, EXP4.B14, JP2.3, SLOT2.B14, SLOT3.B14
- removed net ZBUS15: EXP0.B16, EXP1.B16, EXP4.B16, JP2.1, SLOT2.B16, SLOT3.B16
- removed net ZBUS2: EXP0.A8, EXP1.A8, EXP4.A8, JP2.27, SLOT2.A8, SLOT3.A8
- removed net ZBUS3: EXP0.A10, EXP1.A10, EXP4.A10, JP2.25, SLOT2.A10, SLOT3.A10
- removed net ZBUS4: EXP0.A12, EXP1.A12, EXP4.A12, JP2.23, SLOT2.A12, SLOT3.A12
- removed net ZBUS5: EXP0.A14, EXP1.A14, EXP4.A14, JP2.21, SLOT2.A14, SLOT3.A14
- removed net ZBUS6: EXP0.A16, EXP1.A16, EXP4.A16, JP2.19, SLOT2.A16, SLOT3.A16
- removed net ZBUS7: EXP0.A18, EXP1.A18, EXP4.A18, JP2.17, SLOT2.A18, SLOT3.A18
- removed net ZBUS8: EXP0.B2, EXP1.B2, EXP4.B2, JP2.15, SLOT2.B2, SLOT3.B2
- removed net ZBUS9: EXP0.B4, EXP1.B4, EXP4.B4, JP2.13, SLOT2.B4, SLOT3.B4
- new net !SP1_IRQ!: R4.2, SLOT1.B10
- new net !SPI0_IRQ!: R5.2, SLOT0.B10
- new net !SPI2_IRQ!: R3.2, SLOT2.B10
- new net !SPI3_IRQ!: R2.2, SLOT3.B10
- new net !SPI4_IRQ!: R1.2, SLOT4.B10
- new net A0: SLOT0.A1, SLOT1.A1, SLOT2.A1, SLOT3.A1, SLOT4.A1, U$1.A0@16, U$3.A1
- new net A1: SLOT0.A3, SLOT1.A3, SLOT2.A3, SLOT3.A3, SLOT4.A3, U$1.A1@14, U$3.B1
- new net A10: SLOT0.B3, SLOT1.B3, SLOT2.B3, SLOT3.B3, SLOT4.B3, U$1.A10@46, U$3.A6
- new net A11: SLOT0.B5, SLOT1.B5, SLOT2.B5, SLOT3.B5, SLOT4.B5, U$1.A11@44, U$3.B6
- new net A12: SLOT0.B7, SLOT1.B7, SLOT2.B7, SLOT3.B7, SLOT4.B7, U$1.A12@42, U$3.A7
- new net A13: SLOT0.B9, SLOT1.B9, SLOT2.B9, SLOT3.B9, SLOT4.B9, U$1.A13@40, U$3.B7
- new net A14: SLOT0.B11, SLOT1.B11, SLOT2.B11, SLOT3.B11, SLOT4.B11, U$1.A14@38, U$3.A8
- new net A15: SLOT0.B13, SLOT1.B13, SLOT2.B13, SLOT3.B13, SLOT4.B13, U$1.A15@36, U$3.B8
- new net A2: SLOT0.A5, SLOT1.A5, SLOT2.A5, SLOT3.A5, SLOT4.A5, U$1.A2@12, U$3.A2
- new net A3: SLOT0.A7, SLOT1.A7, SLOT2.A7, SLOT3.A7, SLOT4.A7, U$1.A3@10, U$3.B2
- new net A4: SLOT0.A9, SLOT1.A9, SLOT2.A9, SLOT3.A9, SLOT4.A9, U$1.A4@8, U$3.A3
- new net A5: SLOT0.A11, SLOT1.A11, SLOT2.A11, SLOT3.A11, SLOT4.A11, U$1.A5@6, U$3.B3
- new net A6: SLOT0.A13, SLOT1.A13, SLOT2.A13, SLOT3.A13, SLOT4.A13, U$1.A6@4, U$3.A4
- new net A7: SLOT0.A15, SLOT1.A15, SLOT2.A15, SLOT3.A15, SLOT4.A15, U$1.A7@2, U$3.B4
- new net A8: SLOT0.A17, SLOT1.A17, SLOT2.A17, SLOT3.A17, SLOT4.A17, U$1.A8@50, U$3.A5
- new net A9: SLOT0.B1, SLOT1.B1, SLOT2.B1, SLOT3.B1, SLOT4.B1, U$1.A9@48, U$3.B5
- new net AVALID: SLOT0.B15, SLOT1.B15, SLOT2.B15, SLOT3.B15, SLOT4.B15
- new net D0: SLOT0.A10, SLOT1.A10, SLOT2.A10, SLOT3.A10, SLOT4.A10, U$1.D0@15, U$3.B9
- new net D1: SLOT0.A12, SLOT1.A12, SLOT2.A12, SLOT3.A12, SLOT4.A12, U$1.D1@13, U$3.A10
- new net D2: SLOT0.A14, SLOT1.A14, SLOT2.A14, SLOT3.A14, SLOT4.A14, U$1.D2@11, U$3.B10
- new net D3: SLOT0.A16, SLOT1.A16, SLOT2.A16, SLOT3.A16, SLOT4.A16, U$1.D3@9, U$3.A11
- new net D4: SLOT0.A18, SLOT1.A18, SLOT2.A18, SLOT3.A18, SLOT4.A18, U$1.D4@7, U$3.B11
- new net D5: SLOT0.B2, SLOT1.B2, SLOT2.B2, SLOT3.B2, SLOT4.B2, U$1.D5@5, U$3.A12
- new net D6: SLOT0.B4, SLOT1.B4, SLOT2.B4, SLOT3.B4, SLOT4.B4, U$1.D6@3, U$3.B12
- new net D7: SLOT0.B6, SLOT1.B6, SLOT2.B6, SLOT3.B6, SLOT4.B6, U$1.D7@1, U$3.A13
- new net N$10: LD4.A, R107.2
- new net N$3: LD1.A, R98.2
- new net N$5: LD0.A, R27.2
- new net N$6: R104.1, R64.1, SLOT3.A8
- new net N$7: R101.1, R63.1, SLOT2.A8
- new net N$8: LD3.A, R104.2
- new net N$9: R107.1, R65.1, SLOT4.A8
- new net PRESENT0: R62.1, R98.1, SLOT0.A8
- new net PRESENT1: R27.1, R61.1, SLOT1.A8
- new net SPI0_CLK: SLOT0.B12
- new net SPI0_MISO: SLOT0.B14
- new net SPI0_MOSI: SLOT0.B16
- new net SPI1_CLK: SLOT1.B12
- new net SPI1_MISO: SLOT1.B14
- new net SPI1_MOSI: SLOT1.B16
- new net SPI3_CLK: SLOT3.B12
- new net SPI3_MISO: SLOT3.B14
- new net SPI3_MOSI: SLOT3.B16
- new net SPI4_CLK: SLOT4.B12
- new net SPI4_MISO: SLOT4.B14
- new net SPI4_MOSI: SLOT4.B16
- net +3V3: now also SLOT0.A2, SLOT1.A2, SLOT2.A2, SLOT3.A2, SLOT4.A2; no longer JP2.6, JP2.8
- net +5V: now also C1.1, C56.2, R1.1, R2.1, R3.1, R4.1, R5.1, SLOT0.A4, SLOT0.A6, SLOT1.A4, SLOT1.A6, SLOT2.A4, SLOT2.A6, SLOT3.A4, SLOT3.A6, SLOT4.A4, SLOT4.A6; no longer C54.1, C56.1, JP2.2, JP2.4
- net GND: now also C1.2, C56.1, LD0.C, LD1.C, LD2.C, LD3.C, LD4.C, R61.2, R62.2, R63.2, R64.2, R65.2, SLOT0.B17, SLOT0.B18, SLOT0.B8, SLOT1.B17, SLOT1.B18, SLOT1.B8, SLOT2.B17, SLOT2.B8, SLOT3.B17, SLOT3.B8, SLOT4.B17, SLOT4.B18, SLOT4.B8; no longer C54.2, C56.2, EXP0.B18, EXP1.B18, EXP4.B18, JP2.24, JP2.33, JP2.39, LD_0P1.C, LD_1P.C, LD_2P.C, LD_3P.C, LD_4P.C, R61.1, R62.1, R63.1, R64.1, R65.1
- net N$1: now also LD2.A, R101.2; no longer LD_0P1.A, R27.2
- net SPI2_CLK: now also SLOT2.B12; no longer JP2.10
- net SPI2_MISO: now also SLOT2.B14; no longer JP2.14
- net SPI2_MOSI: now also SLOT2.B16; no longer JP2.18
Other:
- note removed: "+5V Card-present Slot ID"
- note removed: "+5V Slot 3.3v Card-present Slot ID"
- note removed: "B1,2,3 B4 A1,2,3"
- note removed: "B1,2,3 B5,6,7 B4 A1,2,3"
- note removed: "Green and Orange LEDs are configured for 20mA current"
- note removed: "Slot id: 0,0,0"
- note removed: "Slot id: 0,0,1"
- note removed: "Slot id: 0,1,0"
- note removed: "Slot id: 0,1,1"

Commit message: More work on the dual-core STM
Parts:
- removed U1: USD-SOCKETNEW, SparkFun:USD-SOCKETNEW
- added J2: MICROSD_MOLEX_5025700893, j_microsd_molex_5025700893:MICROSD_MOLEX_5025700893
- CN1: USE (none) -> 0471510001
- IC1: USE (none) -> STM32MP157AAA3
- IC2: USE (none) -> IS43TR16256AL-125KBL
- IC3: USE (none) -> TFP410PAP
- IC4: USE (none) -> STPMIC1APQR
- J1: USE (none) -> dc-005
- J3: USE (none) -> RJMG2310228A0ER
- SLOT0, SLOT1, SLOT2, SLOT3, SLOT4: USE (none) -> 10018784-10210TLF
