File: boards/xe-lvl/xe-lvl.sch (EAGLE design)
At the start: 67 parts, among them IC1 STM32MP157AAA3, IC2 MT41K256M16TW-107_P, IC3 STPMIC1APQR, J1 DCJ0202

Commit message: Get the power and DDR parts sorted out. Still needs layout on the DDR.
Parts:
- added C46, C47, C48, C49, C50, C51, C52, C53, C54, C55, C56, C57, C58, C59, C62, C63, C64, C65, C66, C67, C68, C69, C70, C71, C72, C73: 100nF, rcl:C-EUC0201
- added C60, C61: 10uF, rcl:C-EUC0402
- added C74, C75: 22uF, rcl:C-EUC0402
- added R10, R11, R12, R13, R14, R15, R16, R17, R18, R19, R20, R21, R22, R23, R24, R25, R26, R27, R28, R29, R30, R31, R32, R9: 56R, rcl:R-EU_R0201
- added R4, R5: 240R, rcl:R-EU_R0201
- added R6, R7: 10K, rcl:R-EU_R0201
- added R8: 100R, rcl:R-EU_R0201
- added TP1: TPB1,27, testpad:TPB1,27
- IC2: value MT41K256M16TW-107_P -> IS43TR16256B-125KBL; USE (none) -> IS43TR16256B-125KBL
- renumbered A/D to D7
Connections:
- new net N$15: IC1G$2.DDR_ZQ@K22, R4.1
- new net N$16: IC1G$2.DDR_ATO@AA19, TP1.TP
- new net N$17: IC2.ZQ, R5.1
- net !DDR_CAS!: now also R28.1
- net !DDR_CS!: now also R29.1
- net !DDR_RAS!: now also R27.1
- net !DDR_RESET!: now also R7.2
- net !DDR_WE!: now also R31.1
- net +5V: now also J1.1
- net DDR_A0: now also R9.1
- net DDR_A1: now also R10.1
- net DDR_A10: now also R19.1
- net DDR_A11: now also R20.1
- net DDR_A12: now also R21.1
- net DDR_A13: now also R22.1
- net DDR_A14: now also R23.1
- net DDR_A2: now also R11.1
- net DDR_A3: now also R12.1
- net DDR_A4: now also R13.1
- net DDR_A5: now also R14.1
- net DDR_A6: now also R15.1
- net DDR_A7: now also R16.1
- net DDR_A8: now also R17.1
- net DDR_A9: now also R18.1
- net DDR_BA0: now also R24.1
- net DDR_BA1: now also R25.1
- net DDR_BA2: now also R26.1
- net DDR_CKE: now also R30.1, R6.2
- net DDR_CK_N: now also R8.2
- net DDR_CK_P: now also R8.1
- net DDR_ODT: now also R32.1
- net GND: now also C46.2, C47.1, C48.1, C49.1, C50.1, C51.1, C52.1, C53.1, C54.1, C55.1, C56.1, C57.1, C58.1, C59.1, C60.2, C61.2, C62.1, C63.1, C64.1, C65.1, C66.1, C67.1, C68.1, C69.1, C70.1, C71.1, C72.1, C73.1, C74.1, C75.1, J1.2, J1.3, R4.2, R5.2, R6.1, R7.1
- net VDD_DDR: now also C49.2, C50.2, C51.2, C52.2, C53.2, C54.2, C55.2, C56.2, C57.2, C58.2, C59.2, C60.1, C61.1
- net VREF_DDR: now also C46.1, C47.2, C48.2, IC1G$2.DDR__VREF@AB19, IC2.VREFCA, IC2.VREFDQ
- net VTT_DDR: now also C62.2, C63.2, C64.2, C65.2, C66.2, C67.2, C68.2, C69.2, C70.2, C71.2, C72.2, C73.2, C74.2, C75.2, R10.2, R11.2, R12.2, R13.2, R14.2, R15.2, R16.2, R17.2, R18.2, R19.2, R20.2, R21.2, R22.2, R23.2, R24.2, R25.2, R26.2, R27.2, R28.2, R29.2, R30.2, R31.2, R32.2, R9.2
Other:
- note added: "1% resistor"
- note added: "Default output voltages: Which Voltage Rank LDO1 1.8v 0 LDO2 1.8v 0 LDO3 1.8v 0 LDO4 3.3v 3 LDO5 2.9v 2 LDO6 1.0v 0 REFDDR 0.55v 0 BOOST 5.2v n/a BUCK1 1.2v 2 BUCK2 1.1v 0 BUCK3 3.3v 1 BUCK4 3.3v 2"
- note added: "Rank 0: not powered automatically Rank 1: turned on after T+7ms Rank 2: turned on after T+10ms Rank 3: turned on after T+13ms Notes ----- VOUT2 needs to be set to 1.5v LDO3OUT needs to be set to 0.75v"
- moved on the sheet: IC1G$2, IC2, J1
